Commit message: delete useless code

File: rdc_navigation/orne_box_description/urdf/orne_box.gazebo.xacro (robot description, xacro)
@@ -3,5 +3,5 @@
   <xacro:property name="PI" value="3.1415926535897931"/>
   <xacro:arg name="laser_visual" default="true"/>
-  <xacro:arg name="imu_visual"   default="false"/>
+  <!--xacro:arg name="imu_visual"   default="false"/-->
   <gazebo>
     <plugin name="gazebo_ros_control" filename="libgazebo_ros_control.so">
@@ -35,4 +35,5 @@
     <material>Gazebo/Red</material>
   </gazebo>
+<!--
   <gazebo reference="imu_link">
     <sensor type="imu" name="imu">
@@ -42,4 +43,5 @@
     <material>Gazebo/FlatBlack</material>
   </gazebo>
+-->
   <!-- hokuyo -->
   <gazebo reference="hokuyo_link">

File: rdc_navigation/orne_box_description/urdf/orne_box.urdf.xacro (robot description, xacro)
@@ -5,13 +5,4 @@
   <xacro:include filename="$(find orne_box_description)/urdf/orne_box.gazebo.xacro"/>
   <link name="base_link">
-<!--
-    <visual>
-      <origin xyz="0 0 -0.154" rpy="0 0 0"/>
-      <geometry>
-        <mesh filename="package://orne_box_description/meshes/bases/orne_box_base.stl" scale="1 1 1"/>
-      </geometry>
-      <material name="orange"/>
-    </visual>
--->
     <visual>
       <origin xyz="0.090 0 0.1715" rpy="0 0 0"/>
@@ -21,49 +12,4 @@
       <material name="orange"/>
     </visual>
-    <visual>
-      <origin xyz="0.36125 0 0.2625" rpy="0 0 0"/>
-      <geometry>
-        <box size="0.1425 0.404 0.020"/>
-      </geometry>
-      <material name="orange"/>
-    </visual>
-    <visual>
-      <origin xyz="0.35625 0 0.156" rpy="0 0 0"/>
-      <geometry>
-        <box size="0.1325 0.404 0.020"/>
-      </geometry>
-      <material name="orange"/>
-    </visual>
-    <visual>
-      <origin xyz="-0.120 0 0.4815" rpy="0 0 0"/>
-      <geometry>
-        <box size="0.020 0.404 0.822"/>
-      </geometry>
-      <material name="orange"/>
-    </visual>
-    <collision>
-      <origin xyz="0.090 0 0.1715" rpy="0 0 0"/>
-      <geometry>
-        <box size="0.400 0.404 0.202"/>
-      </geometry>
-    </collision>
-    <collision>
-      <origin xyz="0.36125 0 0.2625" rpy="0 0 0"/>
-      <geometry>
-        <box size="0.1425 0.404 0.020"/>
-      </geometry>
-    </collision>
-    <collision>
-      <origin xyz="0.35625 0 0.156" rpy="0 0 0"/>
-      <geometry>
-        <box size="0.1325 0.404 0.020"/>
-      </geometry>
-    </collision>
-    <collision>
-      <origin xyz="-0.120 0 0.4815" rpy="0 0 0"/>
-      <geometry>
-        <box size="0.020 0.404 0.822"/>
-      </geometry>
-    </collision>
     <inertial>
       <origin xyz="0.090 0 0.1715" rpy="0 0 0"/>
@@ -83,12 +29,6 @@
       <origin xyz="0 0 0" rpy="0 0 0"/>
       <geometry>
-        <mesh filename="package://orne_box_description/meshes/wheels/tire.stl" scale="1 1 1"/>
-      </geometry>
-<!--
-      <origin xyz="0 0 0" rpy="0 0 0"/>
-      <geometry>
         <cylinder length="0.045" radius="0.152"/>
       </geometry>
--->
       <material name="white"/>
     </visual>
@@ -116,12 +56,6 @@
       <origin xyz="0 0 0" rpy="0 0 0"/>
       <geometry>
-        <mesh filename="package://orne_box_description/meshes/wheels/tire.stl" scale="1 1 1"/>
-      </geometry>
-<!--
-      <origin xyz="0 0 0" rpy="0 0 0"/>
-      <geometry>
         <cylinder length="0.045" radius="0.152"/>
       </geometry>
--->
       <material name="white"/>
     </visual>
@@ -176,12 +110,14 @@
     </inertial>
   </link>
-  <xacro:include filename="$(find icart_mini_description)/urdf/sensors/imu.urdf.xacro"/>
+  <!--xacro:include filename="$(find icart_mini_description)/urdf/sensors/imu.urdf.xacro"/-->
   <!-- Setting for imu -->
+  <!--
   <xacro:sensor_imu name="imu" parent="base_link" size="0.05 0.05 0.05">
     <origin xyz="0.3 0 0.2445" rpy="0 0 ${-PI/2}"/>
   </xacro:sensor_imu>
+  -->
   <xacro:include filename="$(find icart_mini_description)/urdf/sensors/hokuyo.urdf.xacro"/>
   <xacro:sensor_hokuyo name="hokuyo" parent="base_link">
-    <origin xyz="0.374295 0 0.2185" rpy="${-PI} 0 0"/>
+    <origin xyz="0.374295 0 0.2185" rpy="0 0 0"/>
   </xacro:sensor_hokuyo>
   <transmission name="tran1">
