Commit message: modify URDF

File: rdc_navigation/orne_box_description/urdf/orne_box.urdf.xacro (robot description, xacro)
@@ -21,5 +21,5 @@
     <parent link="base_link"/>
     <child link="wheel_left_link"/>
-    <origin xyz="0.0 0.23075 0.152" rpy="${-PI/2} 0 0"/>
+    <origin xyz="0.0 0.1525 0.075" rpy="${-PI/2} 0 0"/>
     <axis xyz="0 0 1"/>
     <limit effort="100" velocity="100.0"  lower="-5000" upper="5000" />
@@ -29,5 +29,5 @@
       <origin xyz="0 0 0" rpy="0 0 0"/>
       <geometry>
-        <cylinder length="0.045" radius="0.152"/>
+        <cylinder length="0.030" radius="0.075"/>
       </geometry>
       <material name="white"/>
@@ -36,5 +36,5 @@
       <origin xyz="0 0 0" rpy="0 0 0"/>
       <geometry>
-        <cylinder length="0.045" radius="0.152"/>
+        <cylinder length="0.030" radius="0.075"/>
       </geometry>
     </collision>
@@ -48,5 +48,5 @@
     <parent link="base_link"/>
     <child link="wheel_right_link"/>
-    <origin xyz="0.0 -0.23075 0.152" rpy="${-PI/2} 0 0"/>
+    <origin xyz="0.0 -0.1525 0.075" rpy="${-PI/2} 0 0"/>
     <axis xyz="0 0 1"/>
     <limit effort="100" velocity="100.0"  lower="-5000" upper="5000" />
@@ -56,5 +56,5 @@
       <origin xyz="0 0 0" rpy="0 0 0"/>
       <geometry>
-        <cylinder length="0.045" radius="0.152"/>
+        <cylinder length="0.030" radius="0.075"/>
       </geometry>
       <material name="white"/>
@@ -63,5 +63,5 @@
       <origin xyz="0 0 0" rpy="0 0 0"/>
       <geometry>
-        <cylinder length="0.045" radius="0.152"/>
+        <cylinder length="0.030" radius="0.075"/>
       </geometry>
     </collision>

Commit message: URDFの変更

File: rdc_navigation/orne_box_description/urdf/orne_box.urdf.xacro (robot description, xacro)
@@ -6,7 +6,7 @@
   <link name="base_link">
     <visual>
-      <origin xyz="0.090 0 0.1715" rpy="0 0 0"/>
+      <origin xyz="-0.055 0 0.156" rpy="0 0 0"/>
       <geometry>
-        <box size="0.400 0.404 0.202"/>
+        <box size="0.53 0.3840 0.2"/>
       </geometry>
       <material name="orange"/>
@@ -75,7 +75,45 @@
     <parent link="base_link"/>
     <child link="caster_front_link"/>
-    <origin xyz="0.362 0 0.050" rpy="0 0 0"/>
+    <origin xyz="0.21 0 0.050" rpy="0 0 0"/>
   </joint>
   <link name="caster_front_link">
+    <visual>
+      <origin xyz="0 0.150 0" rpy="${PI/2} 0 0"/>
+      <geometry>
+        <cylinder length="0.025" radius="0.050"/>
+      </geometry>
+      <material name="red"/>
+    </visual>
+    <visual>
+      <origin xyz="0 -0.150 0" rpy="${PI/2} 0 0"/>
+      <geometry>
+        <cylinder length="0.025" radius="0.050"/>
+      </geometry>
+      <material name="red"/>
+    </visual>
+    <collision>
+      <origin xyz="0 0.150 0" rpy="${PI/2} 0 0"/>
+      <geometry>
+        <cylinder length="0.025" radius="0.050"/>
+      </geometry>
+    </collision>
+    <collision>
+      <origin xyz="0 -0.150 0" rpy="${PI/2} 0 0"/>
+      <geometry>
+        <cylinder length="0.025" radius="0.050"/>
+      </geometry>
+    </collision>
+    <inertial>
+      <origin xyz="0 0 0" />
+      <mass value="0.2" />
+      <inertia ixx="0.1" ixy="0.0" ixz="0.0" iyy="0.1" iyz="0.0" izz="0.1" />
+    </inertial>
+  </link>
+  <joint name="caster_back_joint" type="fixed">
+    <parent link="base_link"/>
+    <child link="caster_back_link"/>
+    <origin xyz="-0.21 0 0.050" rpy="0 0 0"/>
+  </joint>
+  <link name="caster_back_link">
     <visual>
       <origin xyz="0 0.150 0" rpy="${PI/2} 0 0"/>
@@ -119,5 +157,5 @@
   <xacro:include filename="$(find icart_mini_description)/urdf/sensors/hokuyo.urdf.xacro"/>
   <xacro:sensor_hokuyo name="hokuyo" parent="base_link">
-    <origin xyz="0.374295 0 0.2185" rpy="0 0 0"/>
+    <origin xyz="0.13 0 0.5" rpy="0 0 0"/>
   </xacro:sensor_hokuyo>
   <transmission name="tran1">
