Commit message: orne_or_description

File: orne_or_description/urdf/cit.xacro (robot description, xacro)
@@ -1,5 +1,5 @@
 <?xml version="1.0"?>
 <robot name="cit" xmlns:xacro="http://www.ros.org/wiki/xacro">
-<xacro:include filename="$(find cit_description)/urdf/icart_mini.xacro"/>
+<xacro:include filename="$(find orne_or_description)/urdf/icart_mini.xacro"/>
 <xacro:include filename="$(find icart_mini_description)/urdf/sensors/imu.urdf.xacro"/>
 <xacro:sensor_imu name="imu" parent="base_link" size="0.05 0.05 0.05">
@@ -10,5 +10,5 @@
     <origin xyz="0.343 0 0.1" rpy="3.14 0 0"/>
 </xacro:sensor_hokuyo>
-<xacro:include filename="$(find cit_description)/urdf/kinect.urdf.xacro"/>
+<xacro:include filename="$(find orne_or_description)/urdf/kinect.urdf.xacro"/>
 <xacro:sensor_kinect name="kinect" parent="base_link">
     <origin xyz="0.27 0 1.22" rpy="0 0 0"/>

File: orne_or_description/urdf/kinect.urdf.xacro (robot description, xacro)
@@ -5,5 +5,5 @@
     xmlns:interface="http://playerstage.sourceforge.net/gazebo/xmlschema/#interface"
     xmlns:sensor="http://playerstage.sourceforge.net/gazebo/xmlschema/#sensor">
-    <xacro:include filename="$(find cit_description)/urdf/kinect.gazebo" />
+    <xacro:include filename="$(find orne_or_description)/urdf/kinect.gazebo" />
     <xacro:macro name="sensor_kinect" params="name parent *origin">
         <joint name="kinect_yaw_joint" type="revolute">

File: orne_or_description/urdf/manipulator.urdf (robot description, URDF)
Before this commit: robot manipulator, 18 links, 17 joints
Links:
- link l_elbow_roll_link: geometry collision box size=0.042 0.042 0.180; visual mesh filename=package://orne_or_description/meshes/elbow_roll.stl scale=0.01 0.01 0.01
- link l_hand_left_link: geometry collision mesh filename=package://orne_or_description/meshes/hand_left.stl scale=0.01 0.01 0.01; visual mesh filename=package://orne_or_description/meshes/hand_left.stl scale=0.01 0.01 0.01
- link l_hand_right_link: geometry collision mesh filename=package://orne_or_description/meshes/hand_right.stl scale=0.01 0.01 0.01; visual mesh filename=package://orne_or_description/meshes/hand_right.stl scale=0.01 0.01 0.01
- link l_sholder_pitch_link: geometry collision box size=0.050 0.05 0.032; visual mesh filename=package://orne_or_description/meshes/shoulder_pitch.stl scale=0.01 0.01 0.01
- link l_sholder_roll_link: geometry collision box size=0.042 0.042 0.200; visual mesh filename=package://orne_or_description/meshes/shoulder_roll.stl scale=0.01 0.01 0.01
- link l_wrist_pitch_link: geometry collision box size=0.0330 0.0320 0.0320; visual mesh filename=package://orne_or_description/meshes/wrist_pitch.stl scale=0.01 0.01 0.01
- link l_wrist_roll_link: geometry collision box size=0.0330 0.0320 0.0320; visual mesh filename=package://orne_or_description/meshes/wrist_roll.stl scale=0.01 0.01 0.01
- link l_wrist_yaw_link: geometry collision box size=0.0330 0.0320 0.0320; visual mesh filename=package://orne_or_description/meshes/wrist_yaw.stl scale=0.01 0.01 0.01

File: orne_or_description/urdf/manipulator.urdf.xacro (robot description, xacro)
@@ -90,5 +90,5 @@
       <origin xyz="0 0 0" rpy="0 0 0"/>
       <geometry>
-        <mesh filename="package://cit_description/meshes/shoulder_pitch.stl" scale="0.01 0.01 0.01"/>
+        <mesh filename="package://orne_or_description/meshes/shoulder_pitch.stl" scale="0.01 0.01 0.01"/>
         <!-- <box size="0.0330 0.050 0.0320"/> -->
       </geometry>
@@ -131,5 +131,5 @@
       <origin xyz="0 0 0" rpy="0 0 0"/>
       <geometry>
-        <mesh filename="package://cit_description/meshes/shoulder_roll.stl" scale="0.01 0.01 0.01"/>
+        <mesh filename="package://orne_or_description/meshes/shoulder_roll.stl" scale="0.01 0.01 0.01"/>
       </geometry>
       <material name="blue"/>
@@ -171,5 +171,5 @@
       <origin xyz="0 0 0" rpy="0 0 0"/>
       <geometry>
-        <mesh filename="package://cit_description/meshes/elbow_roll.stl" scale="0.01 0.01 0.01"/>
+        <mesh filename="package://orne_or_description/meshes/elbow_roll.stl" scale="0.01 0.01 0.01"/>
         <!-- <box size="0.0330 0.0320 0.180"/> -->
       </geometry>
@@ -212,5 +212,5 @@
       <origin xyz=" 0 0 0" rpy="0 0 0"/>
       <geometry>
-        <mesh filename="package://cit_description/meshes/wrist_roll.stl" scale="0.01 0.01 0.01"/>
+        <mesh filename="package://orne_or_description/meshes/wrist_roll.stl" scale="0.01 0.01 0.01"/>
         <!-- <box size="0.0330 0.0320 0.0320"/> -->
       </geometry>
@@ -253,5 +253,5 @@
       <origin xyz="0 0 0" rpy="0 0 0"/>
       <geometry>
-        <mesh filename="package://cit_description/meshes/wrist_pitch.stl" scale="0.01 0.01 0.01"/>
+        <mesh filename="package://orne_or_description/meshes/wrist_pitch.stl" scale="0.01 0.01 0.01"/>
         <!-- <box size="0.0330 0.0320 0.0320"/> -->
       </geometry>
@@ -294,5 +294,5 @@
       <origin xyz="0 0 0" rpy="0 0 0"/>
       <geometry>
-        <mesh filename="package://cit_description/meshes/wrist_yaw.stl" scale="0.01 0.01 0.01"/>
+        <mesh filename="package://orne_or_description/meshes/wrist_yaw.stl" scale="0.01 0.01 0.01"/>
       </geometry>
       <material name="blue"/>
@@ -334,12 +334,12 @@
       <origin xyz="0 0 0" rpy="0 0 0"/>
       <geometry>
-        <mesh filename="package://cit_description/meshes/hand_left.stl" scale="0.01 0.01 0.01"/>
-      </geometry>
-      <material name="red"/>
-    </visual>
-    <collision>
-      <origin xyz="0 0 0" rpy="0 0 0"/>
-      <geometry>
-        <mesh filename="package://cit_description/meshes/hand_left.stl" scale="0.01 0.01 0.01"/>
+        <mesh filename="package://orne_or_description/meshes/hand_left.stl" scale="0.01 0.01 0.01"/>
+      </geometry>
+      <material name="red"/>
+    </visual>
+    <collision>
+      <origin xyz="0 0 0" rpy="0 0 0"/>
+      <geometry>
+        <mesh filename="package://orne_or_description/meshes/hand_left.stl" scale="0.01 0.01 0.01"/>
       </geometry>
     </collision>
@@ -375,12 +375,12 @@
       <origin xyz="0 0 0" rpy="0 0 0"/>
       <geometry>
-        <mesh filename="package://cit_description/meshes/hand_right.stl" scale="0.01 0.01 0.01"/>
-      </geometry>
-      <material name="red"/>
-    </visual>
-    <collision>
-      <origin xyz="0 0 0" rpy="0 0 0"/>
-      <geometry>
-        <mesh filename="package://cit_description/meshes/hand_right.stl" scale="0.01 0.01 0.01"/>
+        <mesh filename="package://orne_or_description/meshes/hand_right.stl" scale="0.01 0.01 0.01"/>
+      </geometry>
+      <material name="red"/>
+    </visual>
+    <collision>
+      <origin xyz="0 0 0" rpy="0 0 0"/>
+      <geometry>
+        <mesh filename="package://orne_or_description/meshes/hand_right.stl" scale="0.01 0.01 0.01"/>
       </geometry>
     </collision>
