Commit message: modify urdf of left arm!

File: orne_or_description/urdf/manipulator.urdf (robot description, URDF)
Before this commit: robot manipulator, 18 links, 17 joints
Links:
- link l_elbow_roll_link: geometry collision box size=0.042 0.180 0.042; visual mesh filename=package://orne_or_description/meshes/l_elbow_roll_link.stl
- link l_hand_left_link: geometry collision mesh filename=package://orne_or_description/meshes/l_hand_left_link.stl; visual mesh filename=package://orne_or_description/meshes/l_hand_left_link.stl
- link l_hand_right_link: geometry collision mesh filename=package://orne_or_description/meshes/l_hand_right_link.stl; visual mesh filename=package://orne_or_description/meshes/l_hand_right_link.stl
- link l_sholder_pitch_link: geometry collision box size=0.0320 0.050 0.0320; visual mesh filename=package://orne_or_description/meshes/l_sholder_pitch_link.s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
- link l_sholder_roll_link: geometry collision box size=0.042 0.200 0.042; visual mesh filename=package://orne_or_description/meshes/l_sholder_roll_link.stl
- link l_wrist_pitch_link: geometry collision box size=0.0330 0.0320 0.0320; visual mesh filename=package://orne_or_description/meshes/l_wrist_pitch_link.stl
- link l_wrist_roll_link: geometry collision box size=0.0330 0.0320 0.0320; visual mesh filename=package://orne_or_description/meshes/l_wrist_roll_link.stl
- link l_wrist_yaw_link: geometry collision box size=0.0330 0.0320 0.0320; visual mesh filename=package://orne_or_description/meshes/l_wrist_yaw_link.stl
Joints:
- joint l_elbow_roll_joint: axis 1 0 0 -> 0 0 -1; origin xyz=0 0 -0.271 rpy=0 0 0 -> xyz=0.000 0.2713 0.000
- joint l_hand_left_joint: axis 1 0 0 -> 0 0 1; origin xyz=0 0.0225 -0.083 rpy=0 0 0 -> xyz=-0.0226 0.079 0.000 rpy=0 0 0
- joint l_hand_right_joint: axis -1 0 0 -> 0 0 -1; origin xyz=0 -0.0225 -0.083 rpy=0 0 0 -> xyz=0.0225 0.079 0.000 rpy=0 0 0
- joint l_sholder_pitch_joint: origin xyz=0 0.14 0 rpy=0 1.57 0 -> xyz=0.000 0.100 0.000
- joint l_sholder_roll_joint: axis 1 0 0 -> 0 0 1; origin xyz=0 0.055 0 rpy=1.57 0 0 -> xyz=0.000 0.0563 0.000
- joint l_wrist_pitch_joint: axis 0 -1 0 -> 1 0 0; origin xyz=0 0 -0.054 rpy=0 0 0 -> xyz=0.000 0.054 0.000 rpy=0 0 0
- joint l_wrist_roll_joint: axis 1 0 0 -> 0 0 1; origin xyz=0 -0.042 -0.271 rpy=0 0 0 -> xyz=-0.042 0.2713 0.000
- joint l_wrist_yaw_joint: axis 0 0 1 -> 0 1 0; origin xyz=0 0 -0.0443 rpy=0 0 0 -> xyz=0.000 0.0483 0.000 rpy=0 0 0

Commit message: add right arm

File: orne_or_description/urdf/manipulator.urdf (robot description, URDF)
Before this commit: robot manipulator, 18 links, 17 joints
Links:
- added link r_hand_link, mass 0.5; collision mesh filename=package://orne_or_description/meshes/r_hand_link.stl; visual mesh filename=package://orne_or_description/meshes/r_hand_link.stl
- link l_elbow_roll_link: geometry collision box size=0.042 0.180 0.042; visual mesh filename=package://orne_or_description/meshes/elbow_roll_link.stl
- link l_sholder_pitch_link: geometry collision box size=0.0320 0.050 0.0320; visual mesh filename=package://orne_or_description/meshes/sholder_pitch_link.stl
- link l_sholder_roll_link: geometry collision box size=0.042 0.200 0.042; visual mesh filename=package://orne_or_description/meshes/sholder_roll_link.stl
- link l_wrist_roll_link: geometry collision box size=0.0330 0.0320 0.0320; visual mesh filename=package://orne_or_description/meshes/wrist_roll_link.stl
- link r_elbow_roll_link: geometry collision box size=0.0330 0.0320 0.180; visual mesh filename=package://orne_or_description/meshes/elbow_roll_link.stl
- link r_sholder_pitch_link: geometry collision box size=0.0330 0.05 0.0320; visual mesh filename=package://orne_or_description/meshes/sholder_pitch_link.stl
- link r_sholder_roll_link: geometry collision box size=0.0330 0.0320 0.180; visual mesh filename=package://orne_or_description/meshes/sholder_roll_link.stl
- link r_wrist_pitch_link: geometry collision box size=0.0330 0.0320 0.0320; visual mesh filename=package://orne_or_description/meshes/r_wrist_pitch_link.stl
- link r_wrist_roll_link: geometry collision box size=0.0330 0.0320 0.0320; visual mesh filename=package://orne_or_description/meshes/wrist_roll_link.stl
- link r_wrist_yaw_link: geometry collision box size=0.0330 0.0320 0.0320; visual mesh filename=package://orne_or_description/meshes/r_wrist_yaw_link.stl
- link sholder_link: geometry collision box size=0.0330 0.28 0.0320; visual mesh filename=package://orne_or_description/meshes/shoulder_link.stl
- link spine_link: geometry collision box size=0.0330 0.0520 1.1; visual mesh filename=package://orne_or_description/meshes/body_link.stl
Joints:
- added joint r_hand_joint: type revolute, parent r_wrist_yaw_link, child r_hand_link, origin xyz=0.000 -0.119 0.0295, axis 1 0 0, limit lower=0 upper=1.57 effort=30 velocity=1.571
- joint l_hand_left_joint: origin xyz=-0.0226 0.079 0.000 rpy=0 0 0 -> xyz=-0.0226 0.083 0.000 rpy=0 0 0
- joint l_hand_right_joint: origin xyz=0.0225 0.079 0.000 rpy=0 0 0 -> xyz=0.0225 0.083 0.000 rpy=0 0 0
- joint l_wrist_pitch_joint: origin xyz=0.000 0.054 0.000 rpy=0 0 0 -> xyz=0.000 0.054 0.000
- joint l_wrist_yaw_joint: origin xyz=0.000 0.0483 0.000 rpy=0 0 0 -> xyz=0.000 0.0443 0.000
- joint r_elbow_roll_joint: axis 1 0 0 -> 0 0 1; origin xyz=0 0 -0.180 rpy=0 0 0 -> xyz=0.000 -0.2713 0.000
- joint r_sholder_pitch_joint: origin xyz=0 -0.14 0 rpy=0 1.57 0 -> xyz=0.000 -0.100 0.000
- joint r_sholder_roll_joint: axis 1 0 0 -> 0 0 1; origin xyz=0 -0.05 0 rpy=-1.57 0 0 -> xyz=0.000 -0.0563 0.000
- joint r_wrist_pitch_joint: axis 0 1 0 -> 1 0 0; origin xyz=0 0 -0.05 rpy=0 0 0 -> xyz=0.000 -0.054 0.000
- joint r_wrist_roll_joint: axis 1 0 0 -> 0 0 1; origin xyz=0 0.04 -0.20 rpy=0 0 0 -> xyz=-0.042 -0.2713 0.000
- joint r_wrist_yaw_joint: axis 0 0 1 -> 0 1 0; origin xyz=0 0 -0.05 rpy=0 0 0 -> xyz=0.000 -0.0443 0.000
- joint spine_joint: origin xyz=0 0 0.044 rpy=0 0 0 -> (none)
