Commit message: head_pitch_link -> head_link

File: orne_or_description/urdf/head.urdf.xacro (robot description, xacro)
@@ -36,9 +36,9 @@
             <origin xyz="0.0713 0 0"/>
             <parent link="head_yaw_link"/>
-            <child link="head_pitch_link"/>
+            <child link="head_link"/>
             <axis xyz="0 1 0"/>
             <limit lower="-1.57" upper="1.57" effort="0.5" velocity="6.0"/>
         </joint>
-        <link name="head_pitch_link">
+        <link name="head_link">
             <inertial>
                 <mass value="0.611" />
@@ -49,5 +49,5 @@
                 <origin xyz=" 0 0 0 " rpy="0 0 0" />
                 <geometry>
-                    <mesh filename="package://orne_or_description/meshes/head_pitch_link.stl"/>
+                    <mesh filename="package://orne_or_description/meshes/head_link.stl"/>
                 </geometry>
             </visual>
@@ -61,5 +61,5 @@
         <joint name="camera_joint" type="fixed">
             <origin xyz="0.03 0 0" rpy="0 0 0"/>
-            <parent link="head_pitch_link"/>
+            <parent link="head_link"/>
             <child link="camera_link"/>
         </joint>
@@ -71,30 +71,4 @@
             </inertial>
         </link>
-<!--
-        <joint name="head_joint" type="fixed">
-            <origin xyz="0 0 0" rpy="-1.5707 0 -1.5707" />
-            <parent link="camera_link" />
-            <child link="head_link" />
-        </joint>
-        <link name="head_link">
-            <inertial>
-                <mass value="0.001" />
-                <origin xyz="0 0 0" />
-                <inertia ixx="0.0001" ixy="0.0" ixz="0.0" iyy="0.0001" iyz="0.0" izz="0.0001" />
-            </inertial>
-            <visual>
-                <origin xyz=" 0 0 0 " rpy="0 0 0" />
-                <geometry>
-                    <mesh filename="package://icart_mini_description/meshes/hokuyo.dae"/>
-                </geometry>
-            </visual>
-            <collision>
-                <origin xyz="0.0 0.0 0.0" rpy="0 0 0" />
-                <geometry>
-                    <box size="0.0730 .2760 0.0720"/>
-                </geometry>
-            </collision>
-        </link>
--->
         <transmission name="tran3">
             <type>transmission_interface/SimpleTransmission</type>

File: orne_or_description/urdf/orne_or.urdf.xacro (robot description, xacro)
@@ -7,5 +7,5 @@
     <origin xyz="0.040 0.000 0.137" rpy="0 0 0"/>
 </xacro:manipulator>
-<xacro:sensor_kinect name="kinect" parent="base_link">
+<xacro:sensor_kinect name="head" parent="base_link">
     <origin xyz="0.068 0.0 1.36" rpy="0 0 0"/>
 </xacro:sensor_kinect>
