Commit message: update right arm

File: orne_or_description/urdf/manipulator.urdf.xacro (robot description, xacro)
@@ -29,12 +29,12 @@
     </visual>
     <collision>
-      <origin xyz="0 0 0.55" rpy="0 0 0"/>
-      <geometry>
-        <box size="0.0330 0.0520 1.1"/>
+      <origin xyz="0 0 0.622" rpy="0 0 0"/>
+      <geometry>
+        <box size="0.020 0.040 1.244"/>d
       </geometry>
     </collision>
   </link>
   <joint name="sholder_slider" type="prismatic">
-    <origin xyz="0 0 0.4" rpy="0 0 0"/>
+    <origin xyz="0 0 0.4"/>
     <parent link="spine_link"/>
     <child link="sholder_link"/>
@@ -49,5 +49,4 @@
     </inertial>
     <visual>
-      <origin xyz="0 0 0" rpy="0 0 0"/>
       <geometry>
         <mesh filename="package://orne_or_description/meshes/shoulder_link.stl"/>
@@ -58,7 +57,7 @@
     </visual>
     <collision>
-      <origin xyz="0.0 0.0 0.0" rpy="0 0 0"/>
-      <geometry>
-        <box size="0.0330 0.28 0.0320"/>
+      <origin xyz="0.023 0.000 0.010"/>
+      <geometry>
+        <box size="0.020 0.200 0.040"/>
       </geometry>
     </collision>
@@ -97,10 +96,4 @@
       <material name="red"/>
     </visual>
-    <collision>
-      <origin xyz="0.0 0.025 0.0"/>
-      <geometry>
-        <box size="0.0320 0.050 0.0320"/>
-      </geometry>
-    </collision>
   </link>
   <gazebo reference="l_sholder_pitch_link">
@@ -139,5 +132,5 @@
       <origin xyz="0.000 0.135 0.000"/>
       <geometry>
-        <box size="0.042 0.200 0.042"/>
+        <box size="0.043 0.296 0.043"/>
       </geometry>
     </collision>
@@ -176,7 +169,7 @@
     </visual>
     <collision>
-      <origin xyz="0.000 0.135 0.000"/>
-      <geometry>
-        <box size="0.042 0.180 0.042"/>
+      <origin xyz="-0.042 0.155 0.000"/>
+      <geometry>
+        <box size="0.043 0.256 0.043"/>
       </geometry>
     </collision>
@@ -214,10 +207,4 @@
       <material name="blue"/>
     </visual>
-    <collision>
-      <origin xyz="0.000 0.016 0.000" rpy="0 0 0"/>
-      <geometry>
-        <box size="0.0330 0.0320 0.0320"/>
-      </geometry>
-    </collision>
   </link>
   <gazebo reference="l_wrist_roll_link">
@@ -256,5 +243,5 @@
       <origin xyz="0.000 0.016 0.000"/>
       <geometry>
-        <box size="0.0330 0.0320 0.0320"/>
+        <box size="0.036 0.056 0.032"/>
       </geometry>
     </collision>
@@ -293,7 +280,7 @@
     </visual>
     <collision>
-      <origin xyz="0 0 0"/>
-      <geometry>
-        <box size="0.0330 0.0320 0.0320"/>
+      <origin xyz="0.007 0.044 0.000"/>
+      <geometry>
+        <box size="0.062 0.086 0.040"/>
       </geometry>
     </collision>
@@ -412,10 +399,4 @@
       <material name="red"/>
     </visual>
-    <collision>
-      <origin xyz="0.0 -0.025 0.0" rpy="0 0 0"/>
-      <geometry>
-        <box size="0.0330 0.05 0.0320"/>
-      </geometry>
-    </collision>
   </link>
   <gazebo reference="r_sholder_pitch_link">
@@ -453,7 +434,7 @@
     </visual>
     <collision>
-      <origin xyz="0.0 0.0 -0.09" rpy="0 0 0"/>
-      <geometry>
-        <box size="0.0330 0.0320 0.180"/>
+      <origin xyz="0.000 -0.135 0.000"/>
+      <geometry>
+        <box size="0.043 0.296 0.043"/>
       </geometry>
     </collision>
@@ -493,7 +474,7 @@
     </visual>
     <collision>
-      <origin xyz="0.0 0.04 -0.09" rpy="0 0 0"/>
-      <geometry>
-        <box size="0.0330 0.0320 0.180"/>
+      <origin xyz="-0.042 -0.155 0.000"/>
+      <geometry>
+        <box size="0.043 0.256 0.043"/>
       </geometry>
     </collision>
@@ -532,10 +513,4 @@
       <material name="blue"/>
     </visual>
-    <collision>
-      <origin xyz="0.0 0.0 -0.016" rpy="0 0 0"/>
-      <geometry>
-        <box size="0.0330 0.0320 0.0320"/>
-      </geometry>
-    </collision>
   </link>
   <gazebo reference="r_wrist_roll_link">
@@ -572,7 +547,7 @@
     </visual>
     <collision>
-      <origin xyz="0.0 0.0 -0.016" rpy="0 0 0"/>
-      <geometry>
-        <box size="0.0330 0.0320 0.0320"/>
+      <origin xyz="0.000 -0.016 0.000"/>
+      <geometry>
+        <box size="0.036 0.056 0.032"/>
       </geometry>
     </collision>

Commit message: add r_hand_link

File: orne_or_description/urdf/manipulator.urdf.xacro (robot description, xacro)
@@ -628,5 +628,5 @@
   <transmission name="trans_r_hand">
     <type>transmission_interface/SimpleTransmission</type>
-    <joint name="r_hand_link">
+    <joint name="r_hand_joint">
       <hardwareInterface>PositionJointInterface</hardwareInterface>
     </joint>
@@ -636,9 +636,4 @@
     </actuator>
   </transmission>
-  <gazebo>
-    <plugin name="gazebo_ros_control" filename="libgazebo_ros_control.so">
-      <robotNamespace>/manipulator</robotNamespace>
-    </plugin>
-  </gazebo>
   </xacro:macro>
 </robot>

Commit message: stable simulation

File: orne_or_description/urdf/manipulator.urdf.xacro (robot description, xacro)
@@ -20,5 +20,5 @@
       <mass value="1.73"/>
       <origin xyz="-0.006 0.004 0.625"/>
-      <inertia ixx="0.904597" ixy="0.0" ixz="0.0" iyy="0.904502" iyz="0.0" izz="0.001093"/>
+      <inertia ixx="1.000" ixy="0.0" ixz="0.0" iyy="1.000" iyz="0.0" izz="0.001"/>
     </inertial>
     <visual>
@@ -46,5 +46,5 @@
       <mass value="0.488"/>
       <origin xyz="0.014 0.000 -0.014"/>
-      <inertia ixx="0.002721" ixy="0.0" ixz="0.0" iyy="0.000784" iyz="0.0" izz="0.002332"/>
+      <inertia ixx="0.010" ixy="0.0" ixz="0.0" iyy="0.001" iyz="0.0" izz="0.010"/>
     </inertial>
     <visual>
@@ -88,5 +88,5 @@
       <mass value="0.206"/>
       <origin xyz="0.000 0.022 -0.007"/>
-      <inertia ixx="0.000262" ixy="0.0" ixz="0.0" iyy="0.000117" iyz="0.0" izz="0.000252"/>
+      <inertia ixx="0.001" ixy="0.0" ixz="0.0" iyy="0.001" iyz="0.0" izz="0.001"/>
     </inertial>
     <visual>
@@ -121,5 +121,5 @@
       <mass value="0.207"/>
       <origin xyz="0.000 0.180 0.000"/>
-      <inertia ixx="0.008446" ixy="0.0" ixz="0.0" iyy="0.000073" iyz="0.0" izz="0.008435"/>
+      <inertia ixx="0.010" ixy="0.0" ixz="0.0" iyy="0.001" iyz="0.0" izz="0.010"/>
     </inertial>
     <visual>
@@ -160,5 +160,5 @@
       <mass value="0.220"/>
       <origin xyz="-0.040 0.170 0.000"/>
-      <inertia ixx="0.008452" ixy="0.0" ixz="0.0" iyy="0.000448" iyz="0.0" izz="0.008807"/>
+      <inertia ixx="0.010" ixy="0.0" ixz="0.0" iyy="0.001" iyz="0.0" izz="0.010"/>
     </inertial>
     <visual>
@@ -199,5 +199,5 @@
       <mass value="0.022"/>
       <origin xyz="0.000 0.027 0.000"/>
-      <inertia ixx="0.000023" ixy="0.0" ixz="0.0" iyy="0.000009" iyz="0.0" izz="0.000023"/>
+      <inertia ixx="0.001" ixy="0.0" ixz="0.0" iyy="0.001" iyz="0.0" izz="0.001"/>
     </inertial>
     <visual>
@@ -232,5 +232,5 @@
       <mass value="0.096"/>
       <origin xyz="0.001 0.014 0.000"/>
-      <inertia ixx="0.000049" ixy="0.0" ixz="0.0" iyy="0.000019" iyz="0.0" izz="0.000053"/>
+      <inertia ixx="0.001" ixy="0.0" ixz="0.0" iyy="0.001" iyz="0.0" izz="0.001"/>
     </inertial>
     <visual>
@@ -271,5 +271,5 @@
       <mass value="0.219"/>
       <origin xyz="0.013 0.049 -0.001"/>
-      <inertia ixx="0.000743" ixy="0.0" ixz="0.0" iyy="0.000113" iyz="0.0" izz="0.000802"/>
+      <inertia ixx="0.001" ixy="0.0" ixz="0.0" iyy="0.001" iyz="0.0" izz="0.001"/>
     </inertial>
     <visual>
@@ -310,5 +310,5 @@
       <mass value="0.059"/>
       <origin xyz="-0.001 0.046 0.007"/>
-      <inertia ixx="0.000263" ixy="0.0" ixz="0.0" iyy="0.000041" iyz="0.0" izz="0.000236"/>
+      <inertia ixx="0.001" ixy="0.0" ixz="0.0" iyy="0.001" iyz="0.0" izz="0.001"/>
     </inertial>
     <visual>
@@ -350,5 +350,5 @@
       <mass value="0.058"/>
       <origin xyz="0.001 0.047 0.007"/>
-      <inertia ixx="0.000259" ixy="0.0" ixz="0.0" iyy="0.000039" iyz="0.0" izz="0.000234"/>
+      <inertia ixx="0.001" ixy="0.0" ixz="0.0" iyy="0.001" iyz="0.0" izz="0.001"/>
     </inertial>
     <visual>
@@ -390,5 +390,5 @@
       <mass value="0.206"/>
       <origin xyz="0.000 -0.022 -0.007"/>
-      <inertia ixx="0.000262" ixy="0.0" ixz="0.0" iyy="0.000117" iyz="0.0" izz="0.000252"/>
+      <inertia ixx="0.001" ixy="0.0" ixz="0.0" iyy="0.001" iyz="0.0" izz="0.001"/>
     </inertial>
     <visual>
@@ -424,5 +424,5 @@
       <mass value="0.207"/>
       <origin xyz="0.000 -0.180 0.000"/>
-      <inertia ixx="0.008446" ixy="0.0" ixz="0.0" iyy="0.000074" iyz="0.0" izz="0.008435" />
+      <inertia ixx="0.010" ixy="0.0" ixz="0.0" iyy="0.001" iyz="0.0" izz="0.010" />
     </inertial>
     <visual>
@@ -464,5 +464,5 @@
       <mass value="0.220"/>
       <origin xyz="-0.040 -0.170 0.000"/>
-      <inertia ixx="0.008452" ixy="0.0" ixz="0.0" iyy="0.000448" iyz="0.0" izz="0.008807"/>
+      <inertia ixx="0.010" ixy="0.0" ixz="0.0" iyy="0.001" iyz="0.0" izz="0.010"/>
     </inertial>
     <visual>
@@ -504,5 +504,5 @@
       <mass value="0.022"/>
       <origin xyz="0.000 -0.027 0.000"/>
-      <inertia ixx="0.000023" ixy="0.0" ixz="0.0" iyy="0.000009" iyz="0.0" izz="0.000023"/>
+      <inertia ixx="0.001" ixy="0.0" ixz="0.0" iyy="0.001" iyz="0.0" izz="0.001"/>
     </inertial>
     <visual>
@@ -538,5 +538,5 @@
       <mass value="0.096"/>
       <origin xyz="-0.001 -0.014 0.000"/>
-      <inertia ixx="0.000049" ixy="0.0" ixz="0.0" iyy="0.000019" iyz="0.0" izz="0.000053"/>
+      <inertia ixx="0.001" ixy="0.0" ixz="0.0" iyy="0.001" iyz="0.0" izz="0.001"/>
     </inertial>
     <visual>
@@ -577,5 +577,5 @@
       <mass value="0.262"/>
       <origin xyz="-0.008 -0.075 0.012"/>
-      <inertia ixx="0.002194" ixy="0.0" ixz="0.0" iyy="0.000352" iyz="0.0" izz="0.002089"/>
+      <inertia ixx="0.010" ixy="0.0" ixz="0.0" iyy="0.001" iyz="0.0" izz="0.010"/>
     </inertial>
     <visual>
@@ -612,5 +612,5 @@
       <mass value="0.059"/>
       <origin xyz="-0.001 -0.008 -0.056"/>
-      <inertia ixx="0.000234" ixy="0.0" ixz="0.0" iyy="0.000300" iyz="0.0" izz="0.000082"/>
+      <inertia ixx="0.001" ixy="0.0" ixz="0.0" iyy="0.001" iyz="0.0" izz="0.001"/>
     </inertial>
     <visual>

File: orne_or_description/urdf/orne_or_cart.urdf.xacro (robot description, xacro)
@@ -6,14 +6,14 @@
   <link name="base_link">
     <visual>
-      <origin xyz="-0.055 0 0.156" rpy="0 0 0"/>
+      <origin xyz="0.090 0 0.1715" rpy="0 0 0"/>
       <geometry>
-        <box size="0.53 0.3840 0.2"/>
+        <box size="0.400 0.404 0.202"/>
       </geometry>
       <material name="orange"/>
     </visual>
     <inertial>
-      <origin xyz="0.090 0 0.1715" rpy="0 0 0"/>
+      <origin xyz="0.030 0 0.0" rpy="0 0 0"/>
       <mass value="25.0"/>
-      <inertia ixx="1.0" ixy="0.0" ixz="0.0" iyy="1.0" iyz="0.0" izz="1.0" />
+      <inertia ixx="1.0" ixy="0.0" ixz="0.0" iyy="1.0" iyz="0.0" izz="0.1" />
     </inertial>
   </link>
@@ -75,45 +75,7 @@
     <parent link="base_link"/>
     <child link="caster_front_link"/>
-    <origin xyz="0.21 0 0.050" rpy="0 0 0"/>
+    <origin xyz="0.362 0 0.050" rpy="0 0 0"/>
   </joint>
   <link name="caster_front_link">
-    <visual>
-      <origin xyz="0 0.150 0" rpy="${PI/2} 0 0"/>
-      <geometry>
-        <cylinder length="0.025" radius="0.050"/>
-      </geometry>
-      <material name="red"/>
-    </visual>
-    <visual>
-      <origin xyz="0 -0.150 0" rpy="${PI/2} 0 0"/>
-      <geometry>
-        <cylinder length="0.025" radius="0.050"/>
-      </geometry>
-      <material name="red"/>
-    </visual>
-    <collision>
-      <origin xyz="0 0.150 0" rpy="${PI/2} 0 0"/>
-      <geometry>
-        <cylinder length="0.025" radius="0.050"/>
-      </geometry>
-    </collision>
-    <collision>
-      <origin xyz="0 -0.150 0" rpy="${PI/2} 0 0"/>
-      <geometry>
-        <cylinder length="0.025" radius="0.050"/>
-      </geometry>
-    </collision>
-    <inertial>
-      <origin xyz="0 0 0" />
-      <mass value="0.2" />
-      <inertia ixx="0.1" ixy="0.0" ixz="0.0" iyy="0.1" iyz="0.0" izz="0.1" />
-    </inertial>
-  </link>
-  <joint name="caster_back_joint" type="fixed">
-    <parent link="base_link"/>
-    <child link="caster_back_link"/>
-    <origin xyz="-0.21 0 0.050" rpy="0 0 0"/>
-  </joint>
-  <link name="caster_back_link">
     <visual>
       <origin xyz="0 0.150 0" rpy="${PI/2} 0 0"/>
@@ -157,5 +119,5 @@
   <xacro:include filename="$(find icart_mini_description)/urdf/sensors/hokuyo.urdf.xacro"/>
   <xacro:sensor_hokuyo name="hokuyo" parent="base_link">
-    <origin xyz="0.13 0 0.5" rpy="0 0 0"/>
+    <origin xyz="0.374295 0 0.2185" rpy="0 0 0"/>
   </xacro:sensor_hokuyo>
   <transmission name="tran1">

Commit message: modify rotate direction

File: orne_or_description/urdf/manipulator.urdf.xacro (robot description, xacro)
@@ -81,5 +81,5 @@
     <parent link="sholder_link"/>
     <child link="l_sholder_pitch_link"/>
-    <axis xyz="0 1 0"/>
+    <axis xyz="0 -1 0"/>
     <limit lower="-1" upper="1" effort="30" velocity="1.571"/>
   </joint>
@@ -114,5 +114,5 @@
     <parent link="l_sholder_pitch_link"/>
     <child link="l_sholder_roll_link"/>
-    <axis xyz="0 0 1"/>
+    <axis xyz="0 0 -1"/>
     <limit lower="-1.57" upper="1.57" effort="30" velocity="1.571"/>
   </joint>
@@ -192,5 +192,5 @@
     <parent link="l_elbow_roll_link"/>
     <child link="l_wrist_roll_link"/>
-    <axis xyz="0 0 1"/>
+    <axis xyz="0 0 -1"/>
     <limit lower="-1.57" upper="1.57" effort="30" velocity="1.571"/>
   </joint>
@@ -303,6 +303,6 @@
     <parent link="l_wrist_yaw_link"/>
     <child link="l_hand_left_link"/>
-    <axis xyz="0 0 1"/>
-    <limit lower="0" upper="1.57" effort="30" velocity="1.571"/>
+    <axis xyz="0 0 -1"/>
+    <limit lower="-1.57" upper="0" effort="30" velocity="1.571"/>
   </joint>
   <link name="l_hand_left_link">
@@ -342,5 +342,5 @@
     <parent link="l_wrist_yaw_link"/>
     <child link="l_hand_right_link"/>
-    <axis xyz="0 0 -1"/>
+    <axis xyz="0 0 1"/>
     <mimic joint="l_hand_left_joint" multiplier="1.0" offset="0.0" />
     <limit lower="-3.14" upper="3.14" effort="30" velocity="1.571"/>
@@ -383,5 +383,5 @@
     <parent link="sholder_link"/>
     <child link="r_sholder_pitch_link"/>
-    <axis xyz="0 1 0"/>
+    <axis xyz="0 -1 0"/>
     <limit lower="-1" upper="1" effort="30" velocity="1.571"/>
   </joint>
@@ -531,5 +531,5 @@
     <parent link="r_wrist_roll_link"/>
     <child link="r_wrist_pitch_link"/>
-    <axis xyz="1 0 0"/>
+    <axis xyz="-1 0 0"/>
     <limit lower="-1.57" upper="1.57" effort="30" velocity="1.571"/>
   </joint>
@@ -570,5 +570,5 @@
     <parent link="r_wrist_pitch_link"/>
     <child link="r_wrist_yaw_link"/>
-    <axis xyz="0 1 0"/>
+    <axis xyz="0 -1 0"/>
     <limit lower="-3.14" upper="3.14" effort="30" velocity="1.571"/>
   </joint>

Commit message: 可動域の設定

File: orne_or_description/urdf/manipulator.urdf.xacro (robot description, xacro)
@@ -82,5 +82,5 @@
     <child link="l_sholder_pitch_link"/>
     <axis xyz="0 -1 0"/>
-    <limit lower="-1" upper="1" effort="30" velocity="1.571"/>
+    <limit lower="-5.58" upper="5.58" effort="30" velocity="1.571"/>
   </joint>
   <link name="l_sholder_pitch_link">
@@ -154,5 +154,5 @@
     <child link="l_elbow_roll_link"/>
     <axis xyz="0 0 -1"/>
-    <limit lower="0.0" upper="3.14" effort="30" velocity="1.571"/>
+    <limit lower="-0.69" upper="2.96" effort="30" velocity="1.571"/>
   </joint>
   <link name="l_elbow_roll_link">
@@ -193,5 +193,5 @@
     <child link="l_wrist_roll_link"/>
     <axis xyz="0 0 -1"/>
-    <limit lower="-1.57" upper="1.57" effort="30" velocity="1.571"/>
+    <limit lower="-1.92" upper="1.92" effort="30" velocity="1.571"/>
   </joint>
   <link name="l_wrist_roll_link">
@@ -226,5 +226,5 @@
     <child link="l_wrist_pitch_link"/>
     <axis xyz="1 0 0"/>
-    <limit lower="-1.57" upper="1.57" effort="30" velocity="1.571"/>
+    <limit lower="-1.92" upper="1.92" effort="30" velocity="1.571"/>
   </joint>
   <link name="l_wrist_pitch_link">
@@ -265,5 +265,5 @@
     <child link="l_wrist_yaw_link"/>
     <axis xyz="0 1 0"/>
-    <limit lower="-3.14" upper="3.14" effort="30" velocity="1.571"/>
+    <limit lower="-5.58" upper="5.58" effort="30" velocity="1.571"/>
   </joint>
   <link name="l_wrist_yaw_link">
@@ -384,5 +384,5 @@
     <child link="r_sholder_pitch_link"/>
     <axis xyz="0 -1 0"/>
-    <limit lower="-1" upper="1" effort="30" velocity="1.571"/>
+    <limit lower="-5.58" upper="5.58" effort="30" velocity="1.571"/>
   </joint>
   <link name="r_sholder_pitch_link">
@@ -458,5 +458,5 @@
     <child link="r_elbow_roll_link"/>
     <axis xyz="0 0 1"/>
-    <limit lower="0.0" upper="3.14" effort="30" velocity="1.571"/>
+    <limit lower="-0.7" upper="2.97" effort="30" velocity="1.571"/>
   </joint>
   <link name="r_elbow_roll_link">
@@ -498,5 +498,5 @@
     <child link="r_wrist_roll_link"/>
     <axis xyz="0 0 1"/>
-    <limit lower="-1.57" upper="1.57" effort="30" velocity="1.571"/>
+    <limit lower="-1.92" upper="1.92" effort="30" velocity="1.571"/>
   </joint>
   <link name="r_wrist_roll_link">
@@ -532,5 +532,5 @@
     <child link="r_wrist_pitch_link"/>
     <axis xyz="-1 0 0"/>
-    <limit lower="-1.57" upper="1.57" effort="30" velocity="1.571"/>
+    <limit lower="-1.92" upper="1.92" effort="30" velocity="1.571"/>
   </joint>
   <link name="r_wrist_pitch_link">
@@ -571,5 +571,5 @@
     <child link="r_wrist_yaw_link"/>
     <axis xyz="0 -1 0"/>
-    <limit lower="-3.14" upper="3.14" effort="30" velocity="1.571"/>
+    <limit lower="-5.58" upper="5.58" effort="30" velocity="1.571"/>
   </joint>
   <link name="r_wrist_yaw_link">
@@ -606,5 +606,5 @@
     <child link="r_hand_link"/>
     <axis xyz="1 0 0"/>
-    <limit lower="0" upper="1.57" effort="30" velocity="1.571"/>
+    <limit lower="0" upper="1.74" effort="30" velocity="1.571"/>
   </joint>
   <link name="r_hand_link">

Commit message: change effort

File: orne_or_description/urdf/manipulator.urdf.xacro (robot description, xacro)
@@ -82,5 +82,5 @@
     <child link="l_sholder_pitch_link"/>
     <axis xyz="0 -1 0"/>
-    <limit lower="-5.58" upper="5.58" effort="30" velocity="1.571"/>
+    <limit lower="-5.58" upper="5.58" effort="4.0" velocity="1.571"/>
   </joint>
   <link name="l_sholder_pitch_link">
@@ -115,5 +115,5 @@
     <child link="l_sholder_roll_link"/>
     <axis xyz="0 0 -1"/>
-    <limit lower="-1.57" upper="1.57" effort="30" velocity="1.571"/>
+    <limit lower="-1.57" upper="1.57" effort="4.0" velocity="1.571"/>
   </joint>
   <link name="l_sholder_roll_link">
@@ -154,5 +154,5 @@
     <child link="l_elbow_roll_link"/>
     <axis xyz="0 0 -1"/>
-    <limit lower="-0.69" upper="2.96" effort="30" velocity="1.571"/>
+    <limit lower="-0.69" upper="2.96" effort="2.5" velocity="1.571"/>
   </joint>
   <link name="l_elbow_roll_link">
@@ -193,5 +193,5 @@
     <child link="l_wrist_roll_link"/>
     <axis xyz="0 0 -1"/>
-    <limit lower="-1.92" upper="1.92" effort="30" velocity="1.571"/>
+    <limit lower="-1.92" upper="1.92" effort="2.5" velocity="1.571"/>
   </joint>
   <link name="l_wrist_roll_link">
@@ -226,5 +226,5 @@
     <child link="l_wrist_pitch_link"/>
     <axis xyz="1 0 0"/>
-    <limit lower="-1.92" upper="1.92" effort="30" velocity="1.571"/>
+    <limit lower="-1.92" upper="1.92" effort="2.5" velocity="1.571"/>
   </joint>
   <link name="l_wrist_pitch_link">
@@ -265,5 +265,5 @@
     <child link="l_wrist_yaw_link"/>
     <axis xyz="0 1 0"/>
-    <limit lower="-5.58" upper="5.58" effort="30" velocity="1.571"/>
+    <limit lower="-5.58" upper="5.58" effort="2.5" velocity="1.571"/>
   </joint>
   <link name="l_wrist_yaw_link">
@@ -304,5 +304,5 @@
     <child link="l_hand_left_link"/>
     <axis xyz="0 0 -1"/>
-    <limit lower="-1.57" upper="0" effort="30" velocity="1.571"/>
+    <limit lower="-1.57" upper="0" effort="2.5" velocity="1.571"/>
   </joint>
   <link name="l_hand_left_link">
@@ -344,5 +344,5 @@
     <axis xyz="0 0 1"/>
     <mimic joint="l_hand_left_joint" multiplier="1.0" offset="0.0" />
-    <limit lower="-3.14" upper="3.14" effort="30" velocity="1.571"/>
+    <limit lower="-3.14" upper="3.14" effort="2.5" velocity="1.571"/>
   </joint>
   <link name="l_hand_right_link">
@@ -384,5 +384,5 @@
     <child link="r_sholder_pitch_link"/>
     <axis xyz="0 -1 0"/>
-    <limit lower="-5.58" upper="5.58" effort="30" velocity="1.571"/>
+    <limit lower="-5.58" upper="5.58" effort="4.0" velocity="1.571"/>
   </joint>
   <link name="r_sholder_pitch_link">
@@ -418,5 +418,5 @@
     <child link="r_sholder_roll_link"/>
     <axis xyz="0 0 1"/>
-    <limit lower="-1.57" upper="1.57" effort="30" velocity="1.571"/>
+    <limit lower="-1.57" upper="1.57" effort="4.0" velocity="1.571"/>
   </joint>
   <link name="r_sholder_roll_link">
@@ -458,5 +458,5 @@
     <child link="r_elbow_roll_link"/>
     <axis xyz="0 0 1"/>
-    <limit lower="-0.7" upper="2.97" effort="30" velocity="1.571"/>
+    <limit lower="-0.7" upper="2.97" effort="2.5" velocity="1.571"/>
   </joint>
   <link name="r_elbow_roll_link">
@@ -498,5 +498,5 @@
     <child link="r_wrist_roll_link"/>
     <axis xyz="0 0 1"/>
-    <limit lower="-1.92" upper="1.92" effort="30" velocity="1.571"/>
+    <limit lower="-1.92" upper="1.92" effort="2.5" velocity="1.571"/>
   </joint>
   <link name="r_wrist_roll_link">
@@ -532,5 +532,5 @@
     <child link="r_wrist_pitch_link"/>
     <axis xyz="-1 0 0"/>
-    <limit lower="-1.92" upper="1.92" effort="30" velocity="1.571"/>
+    <limit lower="-1.92" upper="1.92" effort="2.5" velocity="1.571"/>
   </joint>
   <link name="r_wrist_pitch_link">
@@ -571,5 +571,5 @@
     <child link="r_wrist_yaw_link"/>
     <axis xyz="0 -1 0"/>
-    <limit lower="-5.58" upper="5.58" effort="30" velocity="1.571"/>
+    <limit lower="-5.58" upper="5.58" effort="2.5" velocity="1.571"/>
   </joint>
   <link name="r_wrist_yaw_link">
@@ -606,5 +606,5 @@
     <child link="r_hand_link"/>
     <axis xyz="1 0 0"/>
-    <limit lower="0" upper="1.74" effort="30" velocity="1.571"/>
+    <limit lower="0" upper="1.74" effort="2.5" velocity="1.571"/>
   </joint>
   <link name="r_hand_link">

Commit message: change param

File: orne_or_description/urdf/manipulator.urdf.xacro (robot description, xacro)
@@ -82,5 +82,5 @@
     <child link="l_sholder_pitch_link"/>
     <axis xyz="0 -1 0"/>
-    <limit lower="-5.58" upper="5.58" effort="4.0" velocity="1.571"/>
+    <limit lower="-1.39" upper="1.39" effort="4.0" velocity="1.571"/>
   </joint>
   <link name="l_sholder_pitch_link">
@@ -384,5 +384,5 @@
     <child link="r_sholder_pitch_link"/>
     <axis xyz="0 -1 0"/>
-    <limit lower="-5.58" upper="5.58" effort="4.0" velocity="1.571"/>
+    <limit lower="-1.39" upper="1.39" effort="4.0" velocity="1.571"/>
   </joint>
   <link name="r_sholder_pitch_link">
@@ -458,5 +458,5 @@
     <child link="r_elbow_roll_link"/>
     <axis xyz="0 0 1"/>
-    <limit lower="-0.7" upper="2.97" effort="2.5" velocity="1.571"/>
+    <limit lower="-0.69" upper="2.96" effort="2.5" velocity="1.571"/>
   </joint>
   <link name="r_elbow_roll_link">

Commit message: modify moveit[

File: orne_or_description/urdf/manipulator.urdf.xacro (robot description, xacro)
@@ -344,5 +344,5 @@
     <axis xyz="0 0 1"/>
     <mimic joint="l_hand_left_joint" multiplier="1.0" offset="0.0" />
-    <limit lower="-3.14" upper="3.14" effort="2.5" velocity="1.571"/>
+    <limit lower="-1.57" upper="0.0" effort="2.5" velocity="1.571"/>
   </joint>
   <link name="l_hand_right_link">
