Commit message: fix left hand

File: orne_or_description/urdf/manipulator.urdf.xacro (robot description, xacro)
@@ -378,4 +378,11 @@
     </actuator>
   </transmission>
+  <gazebo>
+    <plugin name="gazebo_mimic_joint_control" filename="libroboticsgroup_upatras_gazebo_mimic_joint_plugin.so">
+      <robotNamespace>/manipulator</robotNamespace>
+      <joint>l_hand_left_joint</joint>
+      <mimicJoint>l_hand_right_joint</mimicJoint>
+    </plugin>
+  </gazebo>
   <!--right arm-->
   <joint name="r_sholder_pitch_joint" type="revolute">

Commit message: kinect to head

File: orne_or_description/urdf/manipulator.urdf.xacro (robot description, xacro)
@@ -5,6 +5,4 @@
     xmlns:interface="http://playerstage.sourceforge.net/gazebo/xmlschema/#interface"
     xmlns:sensor="http://playerstage.sourceforge.net/gazebo/xmlschema/#sensor">
-  <xacro:include filename="$(find orne_or_description)/urdf/head.urdf.xacro"/>
-  <xacro:include filename="$(find orne_or_description)/urdf/head.gazebo" />
   <xacro:macro name="manipulator" params="name parent *origin">
   <joint name="spine_joint" type="fixed">
@@ -13,7 +11,4 @@
     <child link="spine_link"/>
   </joint>
-  <xacro:sensor_kinect name="kinect" parent="spine_link">
-    <origin xyz="0.028 0 1.223" rpy="0 0 0"/>
-  </xacro:sensor_kinect>
   <link name="spine_link">
     <inertial>

File: orne_or_description/urdf/orne_or.urdf.xacro (robot description, xacro)
@@ -3,12 +3,10 @@
 <xacro:include filename="$(find orne_or_description)/urdf/orne_or_cart.urdf.xacro"/>
 <xacro:include filename="$(find orne_or_description)/urdf/manipulator.urdf.xacro"/>
+<xacro:include filename="$(find orne_or_description)/urdf/head.urdf.xacro"/>
 <xacro:manipulator name="manipulator" parent="base_link">
     <origin xyz="0.040 0.000 0.137" rpy="0 0 0"/>
 </xacro:manipulator>
-<!--
-<xacro:include filename="$(find orne_or_description)/urdf/head.xacro"/>
 <xacro:sensor_kinect name="kinect" parent="base_link">
-    <origin xyz="0.27 0 1.22" rpy="0 0 0"/>
+    <origin xyz="0.068 0.0 1.36" rpy="0 0 0"/>
 </xacro:sensor_kinect>
--->
 </robot>

Commit message: sholder->shoulder

File: orne_or_description/urdf/manipulator.urdf.xacro (robot description, xacro)
@@ -30,12 +30,12 @@
     </collision>
   </link>
-  <joint name="sholder_slider" type="prismatic">
+  <joint name="shoulder_slider" type="prismatic">
     <origin xyz="0 0 0.4"/>
     <parent link="spine_link"/>
-    <child link="sholder_link"/>
+    <child link="shoulder_link"/>
     <axis xyz="0 0 1"/>
     <limit effort="1000" lower="-0.2" upper="1.4" velocity="1.0"/>
   </joint>
-  <link name="sholder_link">
+  <link name="shoulder_link">
     <inertial>
       <mass value="0.488"/>
@@ -58,13 +58,13 @@
     </collision>
   </link>
-  <gazebo reference="sholder_link">
+  <gazebo reference="shoulder_link">
     <material>Gazebo/Blue</material>
   </gazebo>
-  <transmission name="trans_sholder_slider">
-    <type>transmission_interface/SimpleTransmission</type>
-    <joint name="sholder_slider">
-      <hardwareInterface>PositionJointInterface</hardwareInterface>
-    </joint>
-    <actuator name="motor_sholder_slider">
+  <transmission name="trans_shoulder_slider">
+    <type>transmission_interface/SimpleTransmission</type>
+    <joint name="shoulder_slider">
+      <hardwareInterface>PositionJointInterface</hardwareInterface>
+    </joint>
+    <actuator name="motor_shoulder_slider">
       <hardwareInterface>PositionJointInterface</hardwareInterface>
       <mechanicalReduction>1</mechanicalReduction>
@@ -72,12 +72,12 @@
   </transmission>
   <!--left arm-->
-  <joint name="l_sholder_pitch_joint" type="revolute">
+  <joint name="l_shoulder_pitch_joint" type="revolute">
     <origin xyz="0.000 0.100 0.000"/>
-    <parent link="sholder_link"/>
-    <child link="l_sholder_pitch_link"/>
+    <parent link="shoulder_link"/>
+    <child link="l_shoulder_pitch_link"/>
     <axis xyz="0 -1 0"/>
     <limit lower="-1.39" upper="1.39" effort="4.0" velocity="1.571"/>
   </joint>
-  <link name="l_sholder_pitch_link">
+  <link name="l_shoulder_pitch_link">
     <inertial>
       <mass value="0.206"/>
@@ -87,30 +87,30 @@
     <visual>
       <geometry>
-        <mesh filename="package://orne_or_description/meshes/sholder_pitch_link.stl"/>
-      </geometry>
-      <material name="red"/>
-    </visual>
-  </link>
-  <gazebo reference="l_sholder_pitch_link">
-    <material>Gazebo/Red</material>
-  </gazebo>
-  <transmission name="trans_l_sholder_pitch">
-    <type>transmission_interface/SimpleTransmission</type>
-    <joint name="l_sholder_pitch_joint">
-      <hardwareInterface>PositionJointInterface</hardwareInterface>
-    </joint>
-    <actuator name="motor_l_sholder_pitch">
-      <hardwareInterface>PositionJointInterface</hardwareInterface>
-      <mechanicalReduction>1</mechanicalReduction>
-    </actuator>
-  </transmission>
-  <joint name="l_sholder_roll_joint" type="revolute">
+        <mesh filename="package://orne_or_description/meshes/shoulder_pitch_link.stl"/>
+      </geometry>
+      <material name="red"/>
+    </visual>
+  </link>
+  <gazebo reference="l_shoulder_pitch_link">
+    <material>Gazebo/Red</material>
+  </gazebo>
+  <transmission name="trans_l_shoulder_pitch">
+    <type>transmission_interface/SimpleTransmission</type>
+    <joint name="l_shoulder_pitch_joint">
+      <hardwareInterface>PositionJointInterface</hardwareInterface>
+    </joint>
+    <actuator name="motor_l_shoulder_pitch">
+      <hardwareInterface>PositionJointInterface</hardwareInterface>
+      <mechanicalReduction>1</mechanicalReduction>
+    </actuator>
+  </transmission>
+  <joint name="l_shoulder_roll_joint" type="revolute">
     <origin xyz="0.000 0.0563 0.000"/>
-    <parent link="l_sholder_pitch_link"/>
-    <child link="l_sholder_roll_link"/>
+    <parent link="l_shoulder_pitch_link"/>
+    <child link="l_shoulder_roll_link"/>
     <axis xyz="0 0 -1"/>
     <limit lower="-1.57" upper="1.57" effort="4.0" velocity="1.571"/>
   </joint>
-  <link name="l_sholder_roll_link">
+  <link name="l_shoulder_roll_link">
     <inertial>
       <mass value="0.207"/>
@@ -120,5 +120,5 @@
     <visual>
       <geometry>
-        <mesh filename="package://orne_or_description/meshes/sholder_roll_link.stl"/>
+        <mesh filename="package://orne_or_description/meshes/shoulder_roll_link.stl"/>
       </geometry>
       <material name="blue"/>
@@ -131,13 +131,13 @@
     </collision>
   </link>
-  <gazebo reference="l_sholder_roll_link">
+  <gazebo reference="l_shoulder_roll_link">
     <material>Gazebo/Blue</material>
   </gazebo>
-  <transmission name="trans_l_sholder_roll">
-    <type>transmission_interface/SimpleTransmission</type>
-    <joint name="l_sholder_roll_joint">
-      <hardwareInterface>PositionJointInterface</hardwareInterface>
-    </joint>
-    <actuator name="motor_l_sholder_roll">
+  <transmission name="trans_l_shoulder_roll">
+    <type>transmission_interface/SimpleTransmission</type>
+    <joint name="l_shoulder_roll_joint">
+      <hardwareInterface>PositionJointInterface</hardwareInterface>
+    </joint>
+    <actuator name="motor_l_shoulder_roll">
       <hardwareInterface>PositionJointInterface</hardwareInterface>
       <mechanicalReduction>1</mechanicalReduction>
@@ -146,5 +146,5 @@
   <joint name="l_elbow_roll_joint" type="revolute">
     <origin xyz="0.000 0.2713 0.000"/>
-    <parent link="l_sholder_roll_link"/>
+    <parent link="l_shoulder_roll_link"/>
     <child link="l_elbow_roll_link"/>
     <axis xyz="0 0 -1"/>
@@ -381,12 +381,12 @@
   </gazebo>
   <!--right arm-->
-  <joint name="r_sholder_pitch_joint" type="revolute">
+  <joint name="r_shoulder_pitch_joint" type="revolute">
     <origin xyz="0.000 -0.100 0.000"/>
-    <parent link="sholder_link"/>
-    <child link="r_sholder_pitch_link"/>
+    <parent link="shoulder_link"/>
+    <child link="r_shoulder_pitch_link"/>
     <axis xyz="0 -1 0"/>
     <limit lower="-1.39" upper="1.39" effort="4.0" velocity="1.571"/>
   </joint>
-  <link name="r_sholder_pitch_link">
+  <link name="r_shoulder_pitch_link">
     <inertial>
       <mass value="0.206"/>
@@ -397,30 +397,30 @@
       <origin rpy="0 0 3.14159"/>
       <geometry>
-        <mesh filename="package://orne_or_description/meshes/sholder_pitch_link.stl"/>
-      </geometry>
-      <material name="red"/>
-    </visual>
-  </link>
-  <gazebo reference="r_sholder_pitch_link">
-    <material>Gazebo/Red</material>
-  </gazebo>
-  <transmission name="trans_r_sholder_pitch">
-    <type>transmission_interface/SimpleTransmission</type>
-    <joint name="r_sholder_pitch_joint">
-      <hardwareInterface>PositionJointInterface</hardwareInterface>
-    </joint>
-    <actuator name="motor_r_sholder_pitch">
-      <hardwareInterface>PositionJointInterface</hardwareInterface>
-      <mechanicalReduction>1</mechanicalReduction>
-    </actuator>
-  </transmission>
-  <joint name="r_sholder_roll_joint" type="revolute">
+        <mesh filename="package://orne_or_description/meshes/shoulder_pitch_link.stl"/>
+      </geometry>
+      <material name="red"/>
+    </visual>
+  </link>
+  <gazebo reference="r_shoulder_pitch_link">
+    <material>Gazebo/Red</material>
+  </gazebo>
+  <transmission name="trans_r_shoulder_pitch">
+    <type>transmission_interface/SimpleTransmission</type>
+    <joint name="r_shoulder_pitch_joint">
+      <hardwareInterface>PositionJointInterface</hardwareInterface>
+    </joint>
+    <actuator name="motor_r_shoulder_pitch">
+      <hardwareInterface>PositionJointInterface</hardwareInterface>
+      <mechanicalReduction>1</mechanicalReduction>
+    </actuator>
+  </transmission>
+  <joint name="r_shoulder_roll_joint" type="revolute">
     <origin xyz="0.000 -0.0563 0.000"/>
-    <parent link="r_sholder_pitch_link"/>
-    <child link="r_sholder_roll_link"/>
+    <parent link="r_shoulder_pitch_link"/>
+    <child link="r_shoulder_roll_link"/>
     <axis xyz="0 0 1"/>
     <limit lower="-1.57" upper="1.57" effort="4.0" velocity="1.571"/>
   </joint>
-  <link name="r_sholder_roll_link">
+  <link name="r_shoulder_roll_link">
     <inertial>
       <mass value="0.207"/>
@@ -431,5 +431,5 @@
       <origin rpy="0 0 3.14159"/>
       <geometry>
-        <mesh filename="package://orne_or_description/meshes/sholder_roll_link.stl"/>
+        <mesh filename="package://orne_or_description/meshes/shoulder_roll_link.stl"/>
       </geometry>
       <material name="blue"/>
@@ -442,13 +442,13 @@
     </collision>
   </link>
-  <gazebo reference="r_sholder_roll_link">
+  <gazebo reference="r_shoulder_roll_link">
     <material>Gazebo/Blue</material>
   </gazebo>
-  <transmission name="trans_r_sholder_roll">
-    <type>transmission_interface/SimpleTransmission</type>
-    <joint name="r_sholder_roll_joint">
-      <hardwareInterface>PositionJointInterface</hardwareInterface>
-    </joint>
-    <actuator name="motor_r_sholder_roll">
+  <transmission name="trans_r_shoulder_roll">
+    <type>transmission_interface/SimpleTransmission</type>
+    <joint name="r_shoulder_roll_joint">
+      <hardwareInterface>PositionJointInterface</hardwareInterface>
+    </joint>
+    <actuator name="motor_r_shoulder_roll">
       <hardwareInterface>PositionJointInterface</hardwareInterface>
       <mechanicalReduction>1</mechanicalReduction>
@@ -457,5 +457,5 @@
   <joint name="r_elbow_roll_joint" type="revolute">
     <origin xyz="0.000 -0.2713 0.000"/>
-    <parent link="r_sholder_roll_link"/>
+    <parent link="r_shoulder_roll_link"/>
     <child link="r_elbow_roll_link"/>
     <axis xyz="0 0 1"/>

Commit message: change shoulder height

File: orne_or_description/urdf/manipulator.urdf.xacro (robot description, xacro)
@@ -36,5 +36,5 @@
   </link>
   <joint name="sholder_slider" type="prismatic">
-    <origin xyz="0 0 0.4"/>
+    <origin xyz="0 0 0.66"/>
     <parent link="spine_link"/>
     <child link="sholder_link"/>

Commit message: fix shoulder height

File: orne_or_description/urdf/manipulator.urdf.xacro (robot description, xacro)
@@ -36,5 +36,5 @@
   </link>
   <joint name="sholder_slider" type="prismatic">
-    <origin xyz="0 0 0.66"/>
+    <origin xyz="0 0 0.86"/>
     <parent link="spine_link"/>
     <child link="sholder_link"/>
