Commit message: refine urdf

File: orne_or_description/urdf/kinect.urdf.xacro (robot description, xacro)
@@ -8,5 +8,5 @@
     <xacro:macro name="sensor_kinect" params="name parent *origin">
         <joint name="kinect_yaw_joint" type="revolute">
-            <insert_block  name="origin"/>
+            <xacro:insert_block  name="origin"/>
             <parent link="${parent}"/>
             <child link="kinect_yaw_link"/>
@@ -23,11 +23,9 @@
             </inertial>
             <visual>
-                <origin xyz=" 0 0 0 " rpy="0 0 0" />
                 <geometry>
-                    <box size="0.0330 0.0320 0.0320"/>
+                    <mesh filename="package://orne_or_description/meshes/kinect_yaw_link.stl"/>
                 </geometry>
             </visual>
             <collision>
-                <origin xyz="0.0 0.0 0.0" rpy="0 0 0" />
                 <geometry>
                     <box size="0.0330 0.0320 0.0320"/>
@@ -35,9 +33,10 @@
             </collision>
         </link>
-        <joint name="kinect_pitch_joint" type="fixed">
-            <origin xyz="0.07 0 0" rpy="0 0 0"/>
+        <joint name="kinect_pitch_joint" type="revolute">
+            <origin xyz="0.0713 0 0"/>
             <parent link="kinect_yaw_link"/>
             <child link="kinect_pitch_link"/>
             <axis xyz="0 1 0"/>
+            <limit lower="-1.57" upper="1.57" effort="0.5" velocity="6.0"/>
         </joint>
         <link name="kinect_pitch_link">
@@ -50,5 +49,5 @@
                 <origin xyz=" 0 0 0 " rpy="0 0 0" />
                 <geometry>
-                    <box size="0.0330 0.0320 0.0320"/>
+                    <mesh filename="package://orne_or_description/meshes/kinect_pitch_link.stl"/>
                 </geometry>
             </visual>
@@ -72,4 +71,5 @@
             </inertial>
         </link>
+<!--
         <joint name="kinect_joint" type="fixed">
             <origin xyz="0 0 0" rpy="-1.5707 0 -1.5707" />
@@ -96,4 +96,5 @@
             </collision>
         </link>
+-->
         <transmission name="tran3">
             <type>transmission_interface/SimpleTransmission</type>

File: orne_or_description/urdf/manipulator.urdf.xacro (robot description, xacro)
@@ -5,10 +5,15 @@
     xmlns:interface="http://playerstage.sourceforge.net/gazebo/xmlschema/#interface"
     xmlns:sensor="http://playerstage.sourceforge.net/gazebo/xmlschema/#sensor">
+  <xacro:include filename="$(find orne_or_description)/urdf/kinect.urdf.xacro"/>
+  <xacro:include filename="$(find orne_or_description)/urdf/manipulator.gazebo" />
   <xacro:macro name="manipulator" params="name parent *origin">
   <joint name="spine_joint" type="fixed">
-    <insert_block  name="origin"/>
+    <xacro:insert_block  name="origin"/>
     <parent link="${parent}"/>
     <child link="spine_link"/>
   </joint>
+  <xacro:sensor_kinect name="kinect" parent="spine_link">
+    <origin xyz="0.028 0 1.223" rpy="0 0 0"/>
+  </xacro:sensor_kinect>
   <link name="spine_link">
     <inertial>
@@ -18,7 +23,6 @@
     </inertial>
     <visual>
-      <origin xyz="0 0 0.55" rpy="0 0 0"/>
-      <geometry>
-        <box size="0.0330 0.0520 1.1"/>
+      <geometry>
+        <mesh filename="package://orne_or_description/meshes/body_link.stl"/>
       </geometry>
       <material name="red"/>
@@ -47,5 +51,5 @@
       <origin xyz="0 0 0" rpy="0 0 0"/>
       <geometry>
-        <box size="0.0330 0.28 0.0320"/>
+        <mesh filename="package://orne_or_description/meshes/shoulder_link.stl"/>
       </geometry>
       <material name="blue">
@@ -75,5 +79,5 @@
   <!--left arm-->
   <joint name="l_sholder_pitch_joint" type="revolute">
-    <origin xyz="0 0.14 0" rpy="0 1.57 0"/>
+    <origin xyz="0.000 0.100 0.000"/>
     <parent link="sholder_link"/>
     <child link="l_sholder_pitch_link"/>
@@ -88,15 +92,13 @@
     </inertial>
     <visual>
-      <origin xyz="0 0 0" rpy="0 0 0"/>
-      <geometry>
-        <mesh filename="package://orne_or_description/meshes/shoulder_pitch.stl" scale="0.01 0.01 0.01"/>
-        <!-- <box size="0.0330 0.050 0.0320"/> -->
-      </geometry>
-      <material name="red"/>
-    </visual>
-    <collision>
-      <origin xyz="0.0 0.0 0.0" rpy="0 0 0"/>
-      <geometry>
-        <box size="0.050 0.05 0.032"/>
+      <geometry>
+        <mesh filename="package://orne_or_description/meshes/sholder_pitch_link.stl"/>
+      </geometry>
+      <material name="red"/>
+    </visual>
+    <collision>
+      <origin xyz="0.0 0.025 0.0"/>
+      <geometry>
+        <box size="0.0320 0.050 0.0320"/>
       </geometry>
     </collision>
@@ -116,107 +118,141 @@
   </transmission>
   <joint name="l_sholder_roll_joint" type="revolute">
-    <origin xyz="0 0.055 0" rpy="1.57 0 0"/>
+    <origin xyz="0.000 0.0563 0.000"/>
     <parent link="l_sholder_pitch_link"/>
     <child link="l_sholder_roll_link"/>
+    <axis xyz="0 0 1"/>
+    <limit lower="-1.57" upper="1.57" effort="30" velocity="1.571"/>
+  </joint>
+  <link name="l_sholder_roll_link">
+    <inertial>
+      <mass value="0.5"/>
+      <origin xyz="0 0 0"/>
+      <inertia ixx="1.0" ixy="0.0" ixz="0.0" iyy="1.0" iyz="0.0" izz="1.0"/>
+    </inertial>
+    <visual>
+      <geometry>
+        <mesh filename="package://orne_or_description/meshes/sholder_roll_link.stl"/>
+      </geometry>
+      <material name="blue"/>
+    </visual>
+    <collision>
+      <origin xyz="0.000 0.135 0.000"/>
+      <geometry>
+        <box size="0.042 0.200 0.042"/>
+      </geometry>
+    </collision>
+  </link>
+  <gazebo reference="l_sholder_roll_link">
+    <material>Gazebo/Blue</material>
+  </gazebo>
+  <transmission name="trans_l_sholder_roll">
+    <type>transmission_interface/SimpleTransmission</type>
+    <joint name="l_sholder_roll_joint">
+      <hardwareInterface>PositionJointInterface</hardwareInterface>
+    </joint>
+    <actuator name="motor_l_sholder_roll">
+      <hardwareInterface>PositionJointInterface</hardwareInterface>
+      <mechanicalReduction>1</mechanicalReduction>
+    </actuator>
+  </transmission>
+  <joint name="l_elbow_roll_joint" type="revolute">
+    <origin xyz="0.000 0.2713 0.000"/>
+    <parent link="l_sholder_roll_link"/>
+    <child link="l_elbow_roll_link"/>
+    <axis xyz="0 0 -1"/>
+    <limit lower="0.0" upper="3.14" effort="30" velocity="1.571"/>
+  </joint>
+  <link name="l_elbow_roll_link">
+    <inertial>
+      <mass value="0.5"/>
+      <origin xyz="0 0 0"/>
+      <inertia ixx="1.0" ixy="0.0" ixz="0.0" iyy="1.0" iyz="0.0" izz="1.0"/>
+    </inertial>
+    <visual>
+      <geometry>
+        <mesh filename="package://orne_or_description/meshes/elbow_roll_link.stl"/>
+      </geometry>
+      <material name="red"/>
+    </visual>
+    <collision>
+      <origin xyz="0.000 0.135 0.000"/>
+      <geometry>
+        <box size="0.042 0.180 0.042"/>
+      </geometry>
+    </collision>
+  </link>
+  <gazebo reference="l_elbow_roll_link">
+    <material>Gazebo/Red</material>
+  </gazebo>
+  <transmission name="trans_l_elbow_roll">
+    <type>transmission_interface/SimpleTransmission</type>
+    <joint name="l_elbow_roll_joint">
+      <hardwareInterface>PositionJointInterface</hardwareInterface>
+    </joint>
+    <actuator name="motor_l_elbow_roll">
+      <hardwareInterface>PositionJointInterface</hardwareInterface>
+      <mechanicalReduction>1</mechanicalReduction>
+    </actuator>
+  </transmission>
+  <joint name="l_wrist_roll_joint" type="revolute">
+    <origin xyz="-0.042 0.2713 0.000"/>
+    <parent link="l_elbow_roll_link"/>
+    <child link="l_wrist_roll_link"/>
+    <axis xyz="0 0 1"/>
+    <limit lower="-1.57" upper="1.57" effort="30" velocity="1.571"/>
+  </joint>
+  <link name="l_wrist_roll_link">
+    <inertial>
+      <mass value="0.5"/>
+      <origin xyz="0 0 0"/>
+      <inertia ixx="1.0" ixy="0.0" ixz="0.0" iyy="1.0" iyz="0.0" izz="1.0"/>
+    </inertial>
+    <visual>
+      <geometry>
+        <mesh filename="package://orne_or_description/meshes/wrist_roll_link.stl"/>
+      </geometry>
+      <material name="blue"/>
+    </visual>
+    <collision>
+      <origin xyz="0.000 0.016 0.000" rpy="0 0 0"/>
+      <geometry>
+        <box size="0.0330 0.0320 0.0320"/>
+      </geometry>
+    </collision>
+  </link>
+  <gazebo reference="l_wrist_roll_link">
+    <material>Gazebo/Blue</material>
+  </gazebo>
+  <transmission name="trans_l_wrist_roll">
+    <type>transmission_interface/SimpleTransmission</type>
+    <joint name="l_wrist_roll_joint">
+      <hardwareInterface>PositionJointInterface</hardwareInterface>
+    </joint>
+    <actuator name="motor_l_wrist_roll">
+      <hardwareInterface>PositionJointInterface</hardwareInterface>
+      <mechanicalReduction>1</mechanicalReduction>
+    </actuator>
+  </transmission>
+  <joint name="l_wrist_pitch_joint" type="revolute">
+    <origin xyz="0.000 0.054 0.000"/>
+    <parent link="l_wrist_roll_link"/>
+    <child link="l_wrist_pitch_link"/>
     <axis xyz="1 0 0"/>
     <limit lower="-1.57" upper="1.57" effort="30" velocity="1.571"/>
   </joint>
-  <link name="l_sholder_roll_link">
-    <inertial>
-      <mass value="0.5"/>
-      <origin xyz="0 0 0"/>
-      <inertia ixx="1.0" ixy="0.0" ixz="0.0" iyy="1.0" iyz="0.0" izz="1.0"/>
-    </inertial>
-    <visual>
-      <origin xyz="0 0 0" rpy="0 0 0"/>
-      <geometry>
-        <mesh filename="package://orne_or_description/meshes/shoulder_roll.stl" scale="0.01 0.01 0.01"/>
-      </geometry>
-      <material name="blue"/>
-    </visual>
-    <collision>
-      <origin xyz="0.0 0.0 -0.035" rpy="0 0 0"/>
-      <geometry>
-        <box size="0.042 0.042 0.200"/>
-      </geometry>
-    </collision>
-  </link>
-  <gazebo reference="l_sholder_roll_link">
-    <material>Gazebo/Blue</material>
-  </gazebo>
-  <transmission name="trans_l_sholder_roll">
-    <type>transmission_interface/SimpleTransmission</type>
-    <joint name="l_sholder_roll_joint">
-      <hardwareInterface>PositionJointInterface</hardwareInterface>
-    </joint>
-    <actuator name="motor_l_sholder_roll">
-      <hardwareInterface>PositionJointInterface</hardwareInterface>
-      <mechanicalReduction>1</mechanicalReduction>
-    </actuator>
-  </transmission>
-  <joint name="l_elbow_roll_joint" type="revolute">
-    <origin xyz="0 0 -0.271" rpy="0 0 0"/>
-    <parent link="l_sholder_roll_link"/>
-    <child link="l_elbow_roll_link"/>
-    <axis xyz="1 0 0"/>
-    <limit lower="0.0" upper="3.14" effort="30" velocity="1.571"/>
-  </joint>
-  <link name="l_elbow_roll_link">
-    <inertial>
-      <mass value="0.5"/>
-      <origin xyz="0 0 0"/>
-      <inertia ixx="1.0" ixy="0.0" ixz="0.0" iyy="1.0" iyz="0.0" izz="1.0"/>
-    </inertial>
-    <visual>
-      <origin xyz="0 0 0" rpy="0 0 0"/>
-      <geometry>
-        <mesh filename="package://orne_or_description/meshes/elbow_roll.stl" scale="0.01 0.01 0.01"/>
-        <!-- <box size="0.0330 0.0320 0.180"/> -->
-      </geometry>
-      <material name="red"/>
-    </visual>
-    <collision>
-      <origin xyz="0.0 -0.04 -0.09" rpy="0 0 0"/>
-      <geometry>
-        <box size="0.042 0.042 0.180"/>
-      </geometry>
-    </collision>
-  </link>
-  <gazebo reference="l_elbow_roll_link">
-    <material>Gazebo/Red</material>
-  </gazebo>
-  <transmission name="trans_l_elbow_roll">
-    <type>transmission_interface/SimpleTransmission</type>
-    <joint name="l_elbow_roll_joint">
-      <hardwareInterface>PositionJointInterface</hardwareInterface>
-    </joint>
-    <actuator name="motor_l_elbow_roll">
-      <hardwareInterface>PositionJointInterface</hardwareInterface>
-      <mechanicalReduction>1</mechanicalReduction>
-    </actuator>
-  </transmission>
-  <joint name="l_wrist_roll_joint" type="revolute">
-    <origin xyz="0 -0.042 -0.271" rpy="0 0 0"/>
-    <parent link="l_elbow_roll_link"/>
-    <child link="l_wrist_roll_link"/>
-    <axis xyz="1 0 0"/>
-    <limit lower="-1.57" upper="1.57" effort="30" velocity="1.571"/>
-  </joint>
-  <link name="l_wrist_roll_link">
-    <inertial>
-      <mass value="0.5"/>
-      <origin xyz="0 0 0"/>
-      <inertia ixx="1.0" ixy="0.0" ixz="0.0" iyy="1.0" iyz="0.0" izz="1.0"/>
-    </inertial>
-    <visual>
-      <origin xyz=" 0 0 0" rpy="0 0 0"/>
-      <geometry>
-        <mesh filename="package://orne_or_description/meshes/wrist_roll.stl" scale="0.01 0.01 0.01"/>
-        <!-- <box size="0.0330 0.0320 0.0320"/> -->
-      </geometry>
-      <material name="blue"/>
-    </visual>
-    <collision>
-      <origin xyz="0.0 0.0 -0.016" rpy="0 0 0"/>
+  <link name="l_wrist_pitch_link">
+    <inertial>
+      <mass value="0.5"/>
+      <origin xyz="0 0 0"/>
+      <inertia ixx="1.0" ixy="0.0" ixz="0.0" iyy="1.0" iyz="0.0" izz="1.0"/>
+    </inertial>
+    <visual>
+      <geometry>
+        <mesh filename="package://orne_or_description/meshes/l_wrist_pitch_link.stl"/>
+      </geometry>
+      <material name="red"/>
+    </visual>
+    <collision>
+      <origin xyz="0.000 0.016 0.000"/>
       <geometry>
         <box size="0.0330 0.0320 0.0320"/>
@@ -224,45 +260,4 @@
     </collision>
   </link>
-  <gazebo reference="l_wrist_roll_link">
-    <material>Gazebo/Blue</material>
-  </gazebo>
-  <transmission name="trans_l_wrist_roll">
-    <type>transmission_interface/SimpleTransmission</type>
-    <joint name="l_wrist_roll_joint">
-      <hardwareInterface>PositionJointInterface</hardwareInterface>
-    </joint>
-    <actuator name="motor_l_wrist_roll">
-      <hardwareInterface>PositionJointInterface</hardwareInterface>
-      <mechanicalReduction>1</mechanicalReduction>
-    </actuator>
-  </transmission>
-  <joint name="l_wrist_pitch_joint" type="revolute">
-    <origin xyz="0 0 -0.054" rpy="0 0 0"/>
-    <parent link="l_wrist_roll_link"/>
-    <child link="l_wrist_pitch_link"/>
-    <axis xyz="0 -1 0"/>
-    <limit lower="-1.57" upper="1.57" effort="30" velocity="1.571"/>
-  </joint>
-  <link name="l_wrist_pitch_link">
-    <inertial>
-      <mass value="0.5"/>
-      <origin xyz="0 0 0"/>
-      <inertia ixx="1.0" ixy="0.0" ixz="0.0" iyy="1.0" iyz="0.0" izz="1.0"/>
-    </inertial>
-    <visual>
-      <origin xyz="0 0 0" rpy="0 0 0"/>
-      <geometry>
-        <mesh filename="package://orne_or_description/meshes/wrist_pitch.stl" scale="0.01 0.01 0.01"/>
-        <!-- <box size="0.0330 0.0320 0.0320"/> -->
-      </geometry>
-      <material name="red"/>
-    </visual>
-    <collision>
-      <origin xyz="0.0 0.0 -0.016" rpy="0 0 0"/>
-      <geometry>
-        <box size="0.0330 0.0320 0.0320"/>
-      </geometry>
-    </collision>
-  </link>
   <gazebo reference="l_wrist_pitch_link">
     <material>Gazebo/Red</material>
@@ -279,8 +274,8 @@
   </transmission>
   <joint name="l_wrist_yaw_joint" type="revolute">
-    <origin xyz="0 0 -0.0443" rpy="0 0 0"/>
+    <origin xyz="0.000 0.0443 0.000"/>
     <parent link="l_wrist_pitch_link"/>
     <child link="l_wrist_yaw_link"/>
-    <axis xyz="0 0 1"/>
+    <axis xyz="0 1 0"/>
     <limit lower="-3.14" upper="3.14" effort="30" velocity="1.571"/>
   </joint>
@@ -292,12 +287,11 @@
     </inertial>
     <visual>
-      <origin xyz="0 0 0" rpy="0 0 0"/>
-      <geometry>
-        <mesh filename="package://orne_or_description/meshes/wrist_yaw.stl" scale="0.01 0.01 0.01"/>
+      <geometry>
+        <mesh filename="package://orne_or_description/meshes/l_wrist_yaw_link.stl"/>
       </geometry>
       <material name="blue"/>
     </visual>
     <collision>
-      <origin xyz="0 0 0" rpy="0 0 0"/>
+      <origin xyz="0 0 0"/>
       <geometry>
         <box size="0.0330 0.0320 0.0320"/>
@@ -319,8 +313,8 @@
   </transmission>
   <joint name="l_hand_left_joint" type="revolute">
-    <origin xyz="0 0.0225 -0.083" rpy="0 0 0"/>
+    <origin xyz="-0.0226 0.083 0.000" rpy="0 0 0"/>
     <parent link="l_wrist_yaw_link"/>
     <child link="l_hand_left_link"/>
-    <axis xyz="1 0 0"/>
+    <axis xyz="0 0 1"/>
     <limit lower="0" upper="1.57" effort="30" velocity="1.571"/>
   </joint>
@@ -332,14 +326,13 @@
     </inertial>
     <visual>
+      <geometry>
+        <mesh filename="package://orne_or_description/meshes/l_hand_left_link.stl"/>
+      </geometry>
+      <material name="red"/>
+    </visual>
+    <collision>
       <origin xyz="0 0 0" rpy="0 0 0"/>
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
File: orne_or_description/urdf/orne_or_cart.urdf.xacro (robot description, xacro)
@@ -1,7 +1,7 @@
 <?xml version="1.0" ?>
-<robot name="orne_or" xmlns:xacro="http://www.ros.org/wiki/xacro">
+<robot name="orne_or_cart" xmlns:xacro="http://www.ros.org/wiki/xacro">
   <xacro:property name="PI" value="3.1415926535897931"/>
   <xacro:include filename="$(find icart_mini_description)/urdf/materials.xacro" />
-  <xacro:include filename="$(find orne_or_description)/urdf/orne_or.gazebo.xacro"/>
+  <xacro:include filename="$(find orne_or_description)/urdf/orne_or_cart.gazebo.xacro"/>
   <link name="base_link">
     <visual>
