Commit message: update mass

File: orne_or_description/urdf/kinect.urdf.xacro (robot description, xacro)
@@ -18,7 +18,7 @@
         <link name="kinect_yaw_link">
             <inertial>
-                <mass value="0.001" />
-                <origin xyz="0 0 0" />
-                <inertia ixx="0.0001" ixy="0.0" ixz="0.0" iyy="0.0" iyz="0.0" izz="0.0001" />
+                <mass value="0.107" />
+                <origin xyz="0.053 0.000 0.000" />
+                <inertia ixx="0.000024" ixy="0.0" ixz="0.0" iyy="0.000354" iyz="0.0" izz="0.000355" />
             </inertial>
             <visual>
@@ -42,7 +42,7 @@
         <link name="kinect_pitch_link">
             <inertial>
-                <mass value="0.001" />
-                <origin xyz="0 0 0" />
-                <inertia ixx="0.0001" ixy="0.0" ixz="0.0" iyy="0.0001" iyz="0.0" izz="0.0001" />
+                <mass value="0.611" />
+                <origin xyz="-0.005 0.000 0.045" />
+                <inertia ixx="0.004445" ixy="0.0" ixz="0.0" iyy="0.001536" iyz="0.0" izz="0.003296" />
             </inertial>
             <visual>

File: orne_or_description/urdf/manipulator.urdf.xacro (robot description, xacro)
@@ -18,7 +18,7 @@
   <link name="spine_link">
     <inertial>
-      <mass value="0.5"/>
-      <origin xyz="0 0 0"/>
-      <inertia ixx="1.0" ixy="0.0" ixz="0.0" iyy="1.0" iyz="0.0" izz="1.0"/>
+      <mass value="1.73"/>
+      <origin xyz="-0.006 0.004 0.625"/>
+      <inertia ixx="0.904597" ixy="0.0" ixz="0.0" iyy="0.904502" iyz="0.0" izz="0.001093"/>
     </inertial>
     <visual>
@@ -44,7 +44,7 @@
   <link name="sholder_link">
     <inertial>
-      <mass value="0.5"/>
-      <origin xyz="0 0 0"/>
-      <inertia ixx="1.0" ixy="0.0" ixz="0.0" iyy="1.0" iyz="0.0" izz="1.0"/>
+      <mass value="0.488"/>
+      <origin xyz="0.014 0.000 -0.014"/>
+      <inertia ixx="0.002721" ixy="0.0" ixz="0.0" iyy="0.000784" iyz="0.0" izz="0.002332"/>
     </inertial>
     <visual>
@@ -87,7 +87,7 @@
   <link name="l_sholder_pitch_link">
     <inertial>
-      <mass value="0.5"/>
-      <origin xyz="0 0 0"/>
-      <inertia ixx="1.0" ixy="0.0" ixz="0.0" iyy="1.0" iyz="0.0" izz="1.0"/>
+      <mass value="0.206"/>
+      <origin xyz="0.000 0.022 -0.007"/>
+      <inertia ixx="0.000262" ixy="0.0" ixz="0.0" iyy="0.000117" iyz="0.0" izz="0.000252"/>
     </inertial>
     <visual>
@@ -126,7 +126,7 @@
   <link name="l_sholder_roll_link">
     <inertial>
-      <mass value="0.5"/>
-      <origin xyz="0 0 0"/>
-      <inertia ixx="1.0" ixy="0.0" ixz="0.0" iyy="1.0" iyz="0.0" izz="1.0"/>
+      <mass value="0.207"/>
+      <origin xyz="0.000 0.180 0.000"/>
+      <inertia ixx="0.008446" ixy="0.0" ixz="0.0" iyy="0.000073" iyz="0.0" izz="0.008435"/>
     </inertial>
     <visual>
@@ -165,7 +165,7 @@
   <link name="l_elbow_roll_link">
     <inertial>
-      <mass value="0.5"/>
-      <origin xyz="0 0 0"/>
-      <inertia ixx="1.0" ixy="0.0" ixz="0.0" iyy="1.0" iyz="0.0" izz="1.0"/>
+      <mass value="0.220"/>
+      <origin xyz="-0.040 0.170 0.000"/>
+      <inertia ixx="0.008452" ixy="0.0" ixz="0.0" iyy="0.000448" iyz="0.0" izz="0.008807"/>
     </inertial>
     <visual>
@@ -204,7 +204,7 @@
   <link name="l_wrist_roll_link">
     <inertial>
-      <mass value="0.5"/>
-      <origin xyz="0 0 0"/>
-      <inertia ixx="1.0" ixy="0.0" ixz="0.0" iyy="1.0" iyz="0.0" izz="1.0"/>
+      <mass value="0.022"/>
+      <origin xyz="0.000 0.027 0.000"/>
+      <inertia ixx="0.000023" ixy="0.0" ixz="0.0" iyy="0.000009" iyz="0.0" izz="0.000023"/>
     </inertial>
     <visual>
@@ -243,7 +243,7 @@
   <link name="l_wrist_pitch_link">
     <inertial>
-      <mass value="0.5"/>
-      <origin xyz="0 0 0"/>
-      <inertia ixx="1.0" ixy="0.0" ixz="0.0" iyy="1.0" iyz="0.0" izz="1.0"/>
+      <mass value="0.096"/>
+      <origin xyz="0.001 0.014 0.000"/>
+      <inertia ixx="0.000049" ixy="0.0" ixz="0.0" iyy="0.000019" iyz="0.0" izz="0.000053"/>
     </inertial>
     <visual>
@@ -282,7 +282,7 @@
   <link name="l_wrist_yaw_link">
     <inertial>
-      <mass value="0.5"/>
-      <origin xyz="0 0 0"/>
-      <inertia ixx="1.0" ixy="0.0" ixz="0.0" iyy="1.0" iyz="0.0" izz="1.0"/>
+      <mass value="0.219"/>
+      <origin xyz="0.013 0.049 -0.001"/>
+      <inertia ixx="0.000743" ixy="0.0" ixz="0.0" iyy="0.000113" iyz="0.0" izz="0.000802"/>
     </inertial>
     <visual>
@@ -321,7 +321,7 @@
   <link name="l_hand_left_link">
     <inertial>
-      <mass value="0.5"/>
-      <origin xyz="0 0 0"/>
-      <inertia ixx="1.0" ixy="0.0" ixz="0.0" iyy="1.0" iyz="0.0" izz="1.0"/>
+      <mass value="0.059"/>
+      <origin xyz="-0.001 0.046 0.007"/>
+      <inertia ixx="0.000263" ixy="0.0" ixz="0.0" iyy="0.000041" iyz="0.0" izz="0.000236"/>
     </inertial>
     <visual>
@@ -361,7 +361,7 @@
   <link name="l_hand_right_link">
     <inertial>
-      <mass value="0.5"/>
-      <origin xyz="0 0 0"/>
-      <inertia ixx="1.0" ixy="0.0" ixz="0.0" iyy="1.0" iyz="0.0" izz="1.0"/>
+      <mass value="0.058"/>
+      <origin xyz="0.001 0.047 0.007"/>
+      <inertia ixx="0.000259" ixy="0.0" ixz="0.0" iyy="0.000039" iyz="0.0" izz="0.000234"/>
     </inertial>
     <visual>
@@ -401,7 +401,7 @@
   <link name="r_sholder_pitch_link">
     <inertial>
-      <mass value="0.5"/>
-      <origin xyz="0 0 0"/>
-      <inertia ixx="1.0" ixy="0.0" ixz="0.0" iyy="1.0" iyz="0.0" izz="1.0"/>
+      <mass value="0.206"/>
+      <origin xyz="0.000 -0.022 -0.007"/>
+      <inertia ixx="0.000262" ixy="0.0" ixz="0.0" iyy="0.000117" iyz="0.0" izz="0.000252"/>
     </inertial>
     <visual>
@@ -441,7 +441,7 @@
   <link name="r_sholder_roll_link">
     <inertial>
-      <mass value="0.5"/>
-      <origin xyz="0 0 0"/>
-      <inertia ixx="1.0" ixy="0.0" ixz="0.0" iyy="1.0" iyz="0.0" izz="1.0" />
+      <mass value="0.207"/>
+      <origin xyz="0.000 -0.180 0.000"/>
+      <inertia ixx="0.008446" ixy="0.0" ixz="0.0" iyy="0.000074" iyz="0.0" izz="0.008435" />
     </inertial>
     <visual>
@@ -481,7 +481,7 @@
   <link name="r_elbow_roll_link">
     <inertial>
-      <mass value="0.5"/>
-      <origin xyz="0 0 0"/>
-      <inertia ixx="1.0" ixy="0.0" ixz="0.0" iyy="1.0" iyz="0.0" izz="1.0"/>
+      <mass value="0.220"/>
+      <origin xyz="-0.040 -0.170 0.000"/>
+      <inertia ixx="0.008452" ixy="0.0" ixz="0.0" iyy="0.000448" iyz="0.0" izz="0.008807"/>
     </inertial>
     <visual>
@@ -521,7 +521,7 @@
   <link name="r_wrist_roll_link">
     <inertial>
-      <mass value="0.5"/>
-      <origin xyz="0 0 0"/>
-      <inertia ixx="1.0" ixy="0.0" ixz="0.0" iyy="1.0" iyz="0.0" izz="1.0"/>
+      <mass value="0.022"/>
+      <origin xyz="0.000 -0.027 0.000"/>
+      <inertia ixx="0.000023" ixy="0.0" ixz="0.0" iyy="0.000009" iyz="0.0" izz="0.000023"/>
     </inertial>
     <visual>
@@ -561,7 +561,7 @@
   <link name="r_wrist_pitch_link">
     <inertial>
-      <mass value="0.5"/>
-      <origin xyz="0 0 0"/>
-      <inertia ixx="1.0" ixy="0.0" ixz="0.0" iyy="1.0" iyz="0.0" izz="1.0"/>
+      <mass value="0.096"/>
+      <origin xyz="-0.001 -0.014 0.000"/>
+      <inertia ixx="0.000049" ixy="0.0" ixz="0.0" iyy="0.000019" iyz="0.0" izz="0.000053"/>
     </inertial>
     <visual>
@@ -600,7 +600,7 @@
   <link name="r_wrist_yaw_link">
     <inertial>
-      <mass value="0.5"/>
-      <origin xyz="0 0 0"/>
-      <inertia ixx="1.0" ixy="0.0" ixz="0.0" iyy="1.0" iyz="0.0" izz="1.0"/>
+      <mass value="0.262"/>
+      <origin xyz="-0.008 -0.075 0.012"/>
+      <inertia ixx="0.002194" ixy="0.0" ixz="0.0" iyy="0.000352" iyz="0.0" izz="0.002089"/>
     </inertial>
     <visual>
@@ -611,7 +611,6 @@
     </visual>
     <collision>
-      <origin xyz="0.0 0.0 -0.016"/>
-      <geometry>
-        <box size="0.0330 0.0320 0.0320"/>
+      <geometry>
+        <mesh filename="package://orne_or_description/meshes/r_wrist_yaw_link.stl"/>
       </geometry>
     </collision>
@@ -636,7 +635,7 @@
   <link name="r_hand_link">
     <inertial>
-      <mass value="0.5"/>
-      <origin xyz="0 0 0"/>
-      <inertia ixx="1.0" ixy="0.0" ixz="0.0" iyy="1.0" iyz="0.0" izz="1.0"/>
+      <mass value="0.059"/>
+      <origin xyz="-0.001 -0.008 -0.056"/>
+      <inertia ixx="0.000234" ixy="0.0" ixz="0.0" iyy="0.000300" iyz="0.0" izz="0.000082"/>
     </inertial>
     <visual>

Commit message: rename kinect to head

File: orne_or_description/urdf/kinect.urdf.xacro (robot description, xacro)
@@ -5,10 +5,10 @@
     xmlns:interface="http://playerstage.sourceforge.net/gazebo/xmlschema/#interface"
     xmlns:sensor="http://playerstage.sourceforge.net/gazebo/xmlschema/#sensor">
-    <xacro:include filename="$(find orne_or_description)/urdf/kinect.gazebo" />
+    <xacro:include filename="$(find orne_or_description)/urdf/head.gazebo" />
     <xacro:macro name="sensor_kinect" params="name parent *origin">
-        <joint name="kinect_yaw_joint" type="revolute">
+        <joint name="head_yaw_joint" type="revolute">
             <xacro:insert_block  name="origin"/>
             <parent link="${parent}"/>
-            <child link="kinect_yaw_link"/>
+            <child link="head_yaw_link"/>
             <axis xyz="0 0 1"/>
             <limit lower="-1.57" upper="1.57" effort="0.5" velocity="6.0"/>
@@ -16,5 +16,5 @@
             <dynamics damping="0.4" />
         </joint>
-        <link name="kinect_yaw_link">
+        <link name="head_yaw_link">
             <inertial>
                 <mass value="0.107" />
@@ -24,5 +24,5 @@
             <visual>
                 <geometry>
-                    <mesh filename="package://orne_or_description/meshes/kinect_yaw_link.stl"/>
+                    <mesh filename="package://orne_or_description/meshes/head_yaw_link.stl"/>
                 </geometry>
             </visual>
@@ -33,12 +33,12 @@
             </collision>
         </link>
-        <joint name="kinect_pitch_joint" type="revolute">
+        <joint name="head_pitch_joint" type="revolute">
             <origin xyz="0.0713 0 0"/>
-            <parent link="kinect_yaw_link"/>
-            <child link="kinect_pitch_link"/>
+            <parent link="head_yaw_link"/>
+            <child link="head_pitch_link"/>
             <axis xyz="0 1 0"/>
             <limit lower="-1.57" upper="1.57" effort="0.5" velocity="6.0"/>
         </joint>
-        <link name="kinect_pitch_link">
+        <link name="head_pitch_link">
             <inertial>
                 <mass value="0.611" />
@@ -49,5 +49,5 @@
                 <origin xyz=" 0 0 0 " rpy="0 0 0" />
                 <geometry>
-                    <mesh filename="package://orne_or_description/meshes/kinect_pitch_link.stl"/>
+                    <mesh filename="package://orne_or_description/meshes/head_pitch_link.stl"/>
                 </geometry>
             </visual>
@@ -61,5 +61,5 @@
         <joint name="camera_joint" type="fixed">
             <origin xyz="0.03 0 0" rpy="0 0 0"/>
-            <parent link="kinect_pitch_link"/>
+            <parent link="head_pitch_link"/>
             <child link="camera_link"/>
         </joint>
@@ -72,10 +72,10 @@
         </link>
 <!--
-        <joint name="kinect_joint" type="fixed">
+        <joint name="head_joint" type="fixed">
             <origin xyz="0 0 0" rpy="-1.5707 0 -1.5707" />
             <parent link="camera_link" />
-            <child link="kinect_link" />
+            <child link="head_link" />
         </joint>
-        <link name="kinect_link">
+        <link name="head_link">
             <inertial>
                 <mass value="0.001" />
@@ -99,8 +99,8 @@
         <transmission name="tran3">
             <type>transmission_interface/SimpleTransmission</type>
-            <joint name="kinect_yaw_joint">
+            <joint name="head_yaw_joint">
                 <hardwareInterface>PositionJointInterface</hardwareInterface>
             </joint>
-            <actuator name="kinect_yaw_motor">
+            <actuator name="head_yaw_motor">
                 <hardwareInterface>PositionJointInterface</hardwareInterface>
                 <mechanicalReduction>1</mechanicalReduction>
@@ -109,8 +109,8 @@
         <transmission name="tran4">
             <type>transmission_interface/SimpleTransmission</type>
-            <joint name="kinect_pitch_joint">
+            <joint name="head_pitch_joint">
                 <hardwareInterface>PositionJointInterface</hardwareInterface>
             </joint>
-            <actuator name="kinect_pitch_motor">
+            <actuator name="head_pitch_motor">
                 <hardwareInterface>PositionJointInterface</hardwareInterface>
                 <mechanicalReduction>1</mechanicalReduction>

File: orne_or_description/urdf/manipulator.urdf.xacro (robot description, xacro)
@@ -5,6 +5,6 @@
     xmlns:interface="http://playerstage.sourceforge.net/gazebo/xmlschema/#interface"
     xmlns:sensor="http://playerstage.sourceforge.net/gazebo/xmlschema/#sensor">
-  <xacro:include filename="$(find orne_or_description)/urdf/kinect.urdf.xacro"/>
-  <xacro:include filename="$(find orne_or_description)/urdf/manipulator.gazebo" />
+  <xacro:include filename="$(find orne_or_description)/urdf/head.urdf.xacro"/>
+  <xacro:include filename="$(find orne_or_description)/urdf/head.gazebo" />
   <xacro:macro name="manipulator" params="name parent *origin">
   <joint name="spine_joint" type="fixed">

File: orne_or_description/urdf/orne_or.urdf.xacro (robot description, xacro)
@@ -7,5 +7,5 @@
 </xacro:manipulator>
 <!--
-<xacro:include filename="$(find orne_or_description)/urdf/kinect.urdf.xacro"/>
+<xacro:include filename="$(find orne_or_description)/urdf/head.xacro"/>
 <xacro:sensor_kinect name="kinect" parent="base_link">
     <origin xyz="0.27 0 1.22" rpy="0 0 0"/>

Commit message: feat: 首周りの記述を追加

File: orne_or_description/urdf/kinect.urdf.xacro (robot description, xacro)
@@ -33,4 +33,17 @@
             </collision>
         </link>
+        <gazebo reference="kinect_yaw_link">
+            <material>Gazebo/Blue</material>
+        </gazebo>
+        <transmission name="tran_kinect_yaw_joint">
+            <type>transmission_interface/SimpleTransmission</type>
+            <joint name="kinect_yaw_joint">
+                <hardwareInterface>hardware_interface/PositionJointInterface</hardwareInterface>
+            </joint>
+            <actuator name="motor_kinect_yaw">
+                <hardwareInterface>hardware_interface/PositionJointInterface</hardwareInterface>
+                <mechanicalReduction>1</mechanicalReduction>
+            </actuator>
+        </transmission>
         <joint name="kinect_pitch_joint" type="revolute">
             <origin xyz="0.0713 0 0"/>
@@ -59,4 +72,17 @@
             </collision>
         </link>
+        <gazebo reference="kinect_pitch_link">
+            <material>Gazebo/Red</material>
+        </gazebo>
+        <transmission name="tran_kinect_pitch_joint">
+            <type>transmission_interface/SimpleTransmission</type>
+            <joint name="kinect_pitch_joint">
+                <hardwareInterface>hardware_interface/PositionJointInterface</hardwareInterface>
+            </joint>
+            <actuator name="motor_kinect_pitch">
+                <hardwareInterface>hardware_interface/PositionJointInterface</hardwareInterface>
+                <mechanicalReduction>1</mechanicalReduction>
+            </actuator>
+        </transmission>
         <joint name="camera_joint" type="fixed">
             <origin xyz="0.03 0 0" rpy="0 0 0"/>
@@ -71,5 +97,5 @@
             </inertial>
         </link>
-<!--
+        <!--
         <joint name="kinect_joint" type="fixed">
             <origin xyz="0 0 0" rpy="-1.5707 0 -1.5707" />
@@ -96,25 +122,5 @@
             </collision>
         </link>
--->
-        <transmission name="tran3">
-            <type>transmission_interface/SimpleTransmission</type>
-            <joint name="kinect_yaw_joint">
-                <hardwareInterface>PositionJointInterface</hardwareInterface>
-            </joint>
-            <actuator name="kinect_yaw_motor">
-                <hardwareInterface>PositionJointInterface</hardwareInterface>
-                <mechanicalReduction>1</mechanicalReduction>
-            </actuator>
-        </transmission>
-        <transmission name="tran4">
-            <type>transmission_interface/SimpleTransmission</type>
-            <joint name="kinect_pitch_joint">
-                <hardwareInterface>PositionJointInterface</hardwareInterface>
-            </joint>
-            <actuator name="kinect_pitch_motor">
-                <hardwareInterface>PositionJointInterface</hardwareInterface>
-                <mechanicalReduction>1</mechanicalReduction>
-            </actuator>
-        </transmission>
+        -->
     </xacro:macro>
 </robot>
