Commit message: feat: kinectセンサーのURDFとGazeboプラグインを更新

File: orne_or_description/urdf/arm/manipulator.urdf.xacro (robot description, xacro)
@@ -69,8 +69,8 @@
     <type>transmission_interface/SimpleTransmission</type>
     <joint name="sholder_slider">
-      <hardwareInterface>hardware_interface/PositionJointInterface</hardwareInterface>
+      <hardwareInterface>hardware_interface/EffortJointInterface</hardwareInterface>
     </joint>
     <actuator name="motor_sholder_slider">
-      <hardwareInterface>hardware_interface/PositionJointInterface</hardwareInterface>
+      <hardwareInterface>hardware_interface/EffortJointInterface</hardwareInterface>
       <mechanicalReduction>1</mechanicalReduction>
     </actuator>
@@ -103,8 +103,8 @@
     <type>transmission_interface/SimpleTransmission</type>
     <joint name="l_sholder_pitch_joint">
-      <hardwareInterface>hardware_interface/PositionJointInterface</hardwareInterface>
+      <hardwareInterface>hardware_interface/EffortJointInterface</hardwareInterface>
     </joint>
     <actuator name="motor_l_sholder_pitch">
-      <hardwareInterface>hardware_interface/PositionJointInterface</hardwareInterface>
+      <hardwareInterface>hardware_interface/EffortJointInterface</hardwareInterface>
       <mechanicalReduction>1</mechanicalReduction>
     </actuator>
@@ -142,8 +142,8 @@
     <type>transmission_interface/SimpleTransmission</type>
     <joint name="l_sholder_roll_joint">
-      <hardwareInterface>hardware_interface/PositionJointInterface</hardwareInterface>
+      <hardwareInterface>hardware_interface/EffortJointInterface</hardwareInterface>
     </joint>
     <actuator name="motor_l_sholder_roll">
-      <hardwareInterface>hardware_interface/PositionJointInterface</hardwareInterface>
+      <hardwareInterface>hardware_interface/EffortJointInterface</hardwareInterface>
       <mechanicalReduction>1</mechanicalReduction>
     </actuator>
@@ -181,8 +181,8 @@
     <type>transmission_interface/SimpleTransmission</type>
     <joint name="l_elbow_roll_joint">
-      <hardwareInterface>hardware_interface/PositionJointInterface</hardwareInterface>
+      <hardwareInterface>hardware_interface/EffortJointInterface</hardwareInterface>
     </joint>
     <actuator name="motor_l_elbow_roll">
-      <hardwareInterface>hardware_interface/PositionJointInterface</hardwareInterface>
+      <hardwareInterface>hardware_interface/EffortJointInterface</hardwareInterface>
       <mechanicalReduction>1</mechanicalReduction>
     </actuator>
@@ -214,8 +214,8 @@
     <type>transmission_interface/SimpleTransmission</type>
     <joint name="l_wrist_roll_joint">
-      <hardwareInterface>hardware_interface/PositionJointInterface</hardwareInterface>
+      <hardwareInterface>hardware_interface/EffortJointInterface</hardwareInterface>
     </joint>
     <actuator name="motor_l_wrist_roll">
-      <hardwareInterface>hardware_interface/PositionJointInterface</hardwareInterface>
+      <hardwareInterface>hardware_interface/EffortJointInterface</hardwareInterface>
       <mechanicalReduction>1</mechanicalReduction>
     </actuator>
@@ -253,8 +253,8 @@
     <type>transmission_interface/SimpleTransmission</type>
     <joint name="l_wrist_pitch_joint">
-      <hardwareInterface>hardware_interface/PositionJointInterface</hardwareInterface>
+      <hardwareInterface>hardware_interface/EffortJointInterface</hardwareInterface>
     </joint>
     <actuator name="motor_l_wrist_pitch">
-      <hardwareInterface>hardware_interface/PositionJointInterface</hardwareInterface>
+      <hardwareInterface>hardware_interface/EffortJointInterface</hardwareInterface>
       <mechanicalReduction>1</mechanicalReduction>
     </actuator>
@@ -292,8 +292,8 @@
     <type>transmission_interface/SimpleTransmission</type>
     <joint name="l_wrist_yaw_joint">
-      <hardwareInterface>hardware_interface/PositionJointInterface</hardwareInterface>
+      <hardwareInterface>hardware_interface/EffortJointInterface</hardwareInterface>
     </joint>
     <actuator name="motor_l_wrist_yaw">
-      <hardwareInterface>hardware_interface/PositionJointInterface</hardwareInterface>
+      <hardwareInterface>hardware_interface/EffortJointInterface</hardwareInterface>
       <mechanicalReduction>1</mechanicalReduction>
     </actuator>
@@ -331,8 +331,8 @@
     <type>transmission_interface/SimpleTransmission</type>
     <joint name="l_hand_left_joint">
-      <hardwareInterface>hardware_interface/PositionJointInterface</hardwareInterface>
+      <hardwareInterface>hardware_interface/EffortJointInterface</hardwareInterface>
     </joint>
     <actuator name="motor_l_hand_left">
-      <hardwareInterface>hardware_interface/PositionJointInterface</hardwareInterface>
+      <hardwareInterface>hardware_interface/EffortJointInterface</hardwareInterface>
       <mechanicalReduction>1</mechanicalReduction>
     </actuator>
@@ -371,8 +371,8 @@
     <type>transmission_interface/SimpleTransmission</type>
     <joint name="l_hand_right_joint">
-      <hardwareInterface>hardware_interface/PositionJointInterface</hardwareInterface>
+      <hardwareInterface>hardware_interface/EffortJointInterface</hardwareInterface>
     </joint>
     <actuator name="motor_l_hand_right">
-      <hardwareInterface>hardware_interface/PositionJointInterface</hardwareInterface>
+      <hardwareInterface>hardware_interface/EffortJointInterface</hardwareInterface>
       <mechanicalReduction>1</mechanicalReduction>
     </actuator>
@@ -413,8 +413,8 @@
     <type>transmission_interface/SimpleTransmission</type>
     <joint name="r_sholder_pitch_joint">
-      <hardwareInterface>hardware_interface/PositionJointInterface</hardwareInterface>
+      <hardwareInterface>hardware_interface/EffortJointInterface</hardwareInterface>
     </joint>
     <actuator name="motor_r_sholder_pitch">
-      <hardwareInterface>hardware_interface/PositionJointInterface</hardwareInterface>
+      <hardwareInterface>hardware_interface/EffortJointInterface</hardwareInterface>
       <mechanicalReduction>1</mechanicalReduction>
     </actuator>
@@ -453,8 +453,8 @@
     <type>transmission_interface/SimpleTransmission</type>
     <joint name="r_sholder_roll_joint">
-      <hardwareInterface>hardware_interface/PositionJointInterface</hardwareInterface>
+      <hardwareInterface>hardware_interface/EffortJointInterface</hardwareInterface>
     </joint>
     <actuator name="motor_r_sholder_roll">
-      <hardwareInterface>hardware_interface/PositionJointInterface</hardwareInterface>
+      <hardwareInterface>hardware_interface/EffortJointInterface</hardwareInterface>
       <mechanicalReduction>1</mechanicalReduction>
     </actuator>
@@ -493,8 +493,8 @@
     <type>transmission_interface/SimpleTransmission</type>
     <joint name="r_elbow_roll_joint">
-      <hardwareInterface>hardware_interface/PositionJointInterface</hardwareInterface>
+      <hardwareInterface>hardware_interface/EffortJointInterface</hardwareInterface>
     </joint>
     <actuator name="motor_r_elbow_roll">
-      <hardwareInterface>hardware_interface/PositionJointInterface</hardwareInterface>
+      <hardwareInterface>hardware_interface/EffortJointInterface</hardwareInterface>
       <mechanicalReduction>1</mechanicalReduction>
     </actuator>
@@ -527,8 +527,8 @@
     <type>transmission_interface/SimpleTransmission</type>
     <joint name="r_wrist_roll_joint">
-      <hardwareInterface>hardware_interface/PositionJointInterface</hardwareInterface>
+      <hardwareInterface>hardware_interface/EffortJointInterface</hardwareInterface>
     </joint>
     <actuator name="motor_r_wrist_roll">
-      <hardwareInterface>hardware_interface/PositionJointInterface</hardwareInterface>
+      <hardwareInterface>hardware_interface/EffortJointInterface</hardwareInterface>
       <mechanicalReduction>1</mechanicalReduction>
     </actuator>
@@ -566,8 +566,8 @@
     <type>transmission_interface/SimpleTransmission</type>
     <joint name="r_wrist_pitch_joint">
-      <hardwareInterface>hardware_interface/PositionJointInterface</hardwareInterface>
+      <hardwareInterface>hardware_interface/EffortJointInterface</hardwareInterface>
     </joint>
     <actuator name="motor_r_wrist_pitch">
-      <hardwareInterface>hardware_interface/PositionJointInterface</hardwareInterface>
+      <hardwareInterface>hardware_interface/EffortJointInterface</hardwareInterface>
       <mechanicalReduction>1</mechanicalReduction>
     </actuator>
@@ -601,8 +601,8 @@
     <type>transmission_interface/SimpleTransmission</type>
     <joint name="r_wrist_yaw_joint">
-      <hardwareInterface>hardware_interface/PositionJointInterface</hardwareInterface>
+      <hardwareInterface>hardware_interface/EffortJointInterface</hardwareInterface>
     </joint>
     <actuator name="motor_r_wrist_yaw">
-      <hardwareInterface>hardware_interface/PositionJointInterface</hardwareInterface>
+      <hardwareInterface>hardware_interface/EffortJointInterface</hardwareInterface>
       <mechanicalReduction>1</mechanicalReduction>
     </actuator>
@@ -636,8 +636,8 @@
     <type>transmission_interface/SimpleTransmission</type>
     <joint name="r_hand_joint">
-      <hardwareInterface>hardware_interface/PositionJointInterface</hardwareInterface>
+      <hardwareInterface>hardware_interface/EffortJointInterface</hardwareInterface>
     </joint>
     <actuator name="motor_r_hand">
-      <hardwareInterface>hardware_interface/PositionJointInterface</hardwareInterface>
+      <hardwareInterface>hardware_interface/EffortJointInterface</hardwareInterface>
       <mechanicalReduction>1</mechanicalReduction>
     </actuator>

File: orne_or_description/urdf/cart/orne_or_cart.gazebo.xacro (robot description, xacro)
@@ -7,4 +7,6 @@
     <plugin name="gazebo_ros_control" filename="libgazebo_ros_control.so">
       <robotSimType>icart_mini_gazebo/ICartMiniHWSim</robotSimType>
+      <robotSimType>gazebo_ros_control/DefaultRobotHWSim</robotSimType>
+      <legacyModeNS>true</legacyModeNS>
     </plugin>
   </gazebo>

File: orne_or_description/urdf/orne_or.urdf.xacro (robot description, xacro)
@@ -6,9 +6,3 @@
     <origin xyz="0.040 0.000 0.137" rpy="0 0 0"/>
 </xacro:manipulator>
-<!--
-<xacro:include filename="$(find orne_or_description)/urdf/kinect.urdf.xacro"/>
-<xacro:sensor_kinect name="kinect" parent="base_link">
-    <origin xyz="0.27 0 1.22" rpy="0 0 0"/>
-</xacro:sensor_kinect>
--->
 </robot>

File: orne_or_description/urdf/sensor/kinect.urdf.xacro (robot description, xacro)
@@ -39,8 +39,8 @@
             <type>transmission_interface/SimpleTransmission</type>
             <joint name="kinect_yaw_joint">
-                <hardwareInterface>hardware_interface/PositionJointInterface</hardwareInterface>
+                <hardwareInterface>hardware_interface/EffortJointInterface</hardwareInterface>
             </joint>
             <actuator name="motor_kinect_yaw">
-                <hardwareInterface>hardware_interface/PositionJointInterface</hardwareInterface>
+                <hardwareInterface>hardware_interface/EffortJointInterface</hardwareInterface>
                 <mechanicalReduction>1</mechanicalReduction>
             </actuator>
@@ -78,8 +78,8 @@
             <type>transmission_interface/SimpleTransmission</type>
             <joint name="kinect_pitch_joint">
-                <hardwareInterface>hardware_interface/PositionJointInterface</hardwareInterface>
+                <hardwareInterface>hardware_interface/EffortJointInterface</hardwareInterface>
             </joint>
             <actuator name="motor_kinect_pitch">
-                <hardwareInterface>hardware_interface/PositionJointInterface</hardwareInterface>
+                <hardwareInterface>hardware_interface/EffortJointInterface</hardwareInterface>
                 <mechanicalReduction>1</mechanicalReduction>
             </actuator>
@@ -97,30 +97,4 @@
             </inertial>
         </link>
-        <!--
-        <joint name="kinect_joint" type="fixed">
-            <origin xyz="0 0 0" rpy="-1.5707 0 -1.5707" />
-            <parent link="camera_link" />
-            <child link="kinect_link" />
-        </joint>
-        <link name="kinect_link">
-            <inertial>
-                <mass value="0.001" />
-                <origin xyz="0 0 0" />
-                <inertia ixx="0.0001" ixy="0.0" ixz="0.0" iyy="0.0001" iyz="0.0" izz="0.0001" />
-            </inertial>
-            <visual>
-                <origin xyz=" 0 0 0 " rpy="0 0 0" />
-                <geometry>
-                    <mesh filename="package://icart_mini_description/meshes/hokuyo.dae"/>
-                </geometry>
-            </visual>
-            <collision>
-                <origin xyz="0.0 0.0 0.0" rpy="0 0 0" />
-                <geometry>
-                    <box size="0.0730 .2760 0.0720"/>
-                </geometry>
-            </collision>
-        </link>
-        -->
     </xacro:macro>
 </robot>
