Commit message: fix: 不要なrobotSimTypeを削除し、IMUセンサーの設定をコメントアウト

File: orne_or_description/urdf/cart/orne_or_cart.gazebo.xacro (robot description, xacro)
@@ -7,5 +7,4 @@
     <plugin name="gazebo_ros_control" filename="libgazebo_ros_control.so">
       <robotSimType>icart_mini_gazebo/ICartMiniHWSim</robotSimType>
-      <robotSimType>gazebo_ros_control/DefaultRobotHWSim</robotSimType>
       <legacyModeNS>true</legacyModeNS>
     </plugin>
@@ -37,13 +36,4 @@
     <material>Gazebo/Red</material>
   </gazebo>
-<!--
-  <gazebo reference="imu_link">
-    <sensor type="imu" name="imu">
-      <always_on>true</always_on>
-      <visualize>$(arg imu_visual)</visualize>
-    </sensor>
-    <material>Gazebo/FlatBlack</material>
-  </gazebo>
--->
   <!-- hokuyo -->
   <gazebo reference="hokuyo_link">
