Commit message: feat: トランスミッションを別ファイルに分離し、インターフェースを更新

File: orne_or_description/urdf/cart/orne_or_cart.urdf.xacro (robot description, xacro)
@@ -3,5 +3,7 @@
   <xacro:property name="PI" value="3.1415926535897931"/>
   <xacro:include filename="$(find icart_mini_description)/urdf/materials.xacro" />
+  <xacro:include filename="$(find icart_mini_description)/urdf/sensors/imu.urdf.xacro"/>
   <xacro:include filename="$(find orne_or_description)/urdf/cart/orne_or_cart.gazebo.xacro"/>
+  <xacro:include filename="$(find orne_or_description)/urdf/cart/orne_or_cart.transmission.xacro"/>
   <link name="base_link">
     <visual>
@@ -110,5 +112,4 @@
     </inertial>
   </link>
-  <xacro:include filename="$(find icart_mini_description)/urdf/sensors/imu.urdf.xacro"/>
   <!-- Setting for imu -->
   <xacro:sensor_imu name="imu" parent="base_link" size="0.05 0.05 0.05">
@@ -119,23 +120,3 @@
     <origin xyz="0.374295 0 0.2185" rpy="0 0 0"/>
   </xacro:sensor_hokuyo>
-  <transmission name="tran1">
-    <type>transmission_interface/SimpleTransmission</type>
-    <joint name="left_wheel_hinge">
-      <hardwareInterface>VelocityJointInterface</hardwareInterface>
-    </joint>
-  <actuator name="left_motor">
-      <hardwareInterface>VelocityJointInterface</hardwareInterface>
-      <mechanicalReduction>1</mechanicalReduction>
-    </actuator>
-  </transmission>
-  <transmission name="tran2">
-    <type>transmission_interface/SimpleTransmission</type>
-    <joint name="right_wheel_hinge">
-      <hardwareInterface>VelocityJointInterface</hardwareInterface>
-    </joint>
-  <actuator name="right_motor">
-      <hardwareInterface>VelocityJointInterface</hardwareInterface>
-      <mechanicalReduction>1</mechanicalReduction>
-    </actuator>
-  </transmission>
 </robot>

File: orne_or_description/urdf/orne_or.urdf.xacro (robot description, xacro)
@@ -7,3 +7,4 @@
 </xacro:manipulator>
 <xacro:manipulator_transmission interface="hardware_interface/PositionJointInterface"/>
+<xacro:orne_or_cart_transmission interface="hardware_interface/VelocityJointInterface"/>
 </robot>

Commit message: feat: base_linkとキャスター,IMU,LiDARを修正

File: orne_or_description/urdf/cart/orne_or_cart.urdf.xacro (robot description, xacro)
@@ -6,12 +6,6 @@
   <xacro:include filename="$(find orne_or_description)/urdf/cart/orne_or_cart.gazebo.xacro"/>
   <xacro:include filename="$(find orne_or_description)/urdf/cart/orne_or_cart.transmission.xacro"/>
+  <!-- Base -->
   <link name="base_link">
-    <visual>
-      <origin xyz="0.090 0 0.1715" rpy="0 0 0"/>
-      <geometry>
-        <box size="0.400 0.404 0.202"/>
-      </geometry>
-      <material name="orange"/>
-    </visual>
     <inertial>
       <origin xyz="0.030 0 0.0" rpy="0 0 0"/>
@@ -19,5 +13,18 @@
       <inertia ixx="1.0" ixy="0.0" ixz="0.0" iyy="1.0" iyz="0.0" izz="0.1" />
     </inertial>
+    <visual>
+        <geometry>
+          <mesh filename="package://orne_or_description/meshes/bases/base_link.stl"/>
+        </geometry>
+        <material name="orange"/>
+    </visual>
+    <collision>
+      <origin xyz="0.090 0 0.1715" rpy="0 0 0"/>
+      <geometry>
+        <box size="0.400 0.404 0.202"/>
+      </geometry>
+    </collision>
   </link>
+  <!-- Left Wheel -->
   <joint name="left_wheel_hinge" type="revolute">
     <parent link="base_link"/>
@@ -47,4 +54,5 @@
     </inertial>
   </link>
+  <!-- Right Wheel -->
   <joint name="right_wheel_hinge" type="revolute">
     <parent link="base_link"/>
@@ -74,8 +82,9 @@
     </inertial>
   </link>
+  <!-- Caster -->
   <joint name="caster_front_joint" type="fixed">
     <parent link="base_link"/>
     <child link="caster_front_link"/>
-    <origin xyz="0.362 0 0.050" rpy="0 0 0"/>
+    <origin xyz="-0.3 0 0.050" rpy="0 0 0"/>
   </joint>
   <link name="caster_front_link">
@@ -112,11 +121,8 @@
     </inertial>
   </link>
-  <!-- Setting for imu -->
-  <xacro:sensor_imu name="imu" parent="base_link" size="0.05 0.05 0.05">
-    <origin xyz="0.3 0 0.2445" rpy="0 0 ${-PI/2}"/>
-  </xacro:sensor_imu>
+  <!-- LiDAR -->
   <xacro:include filename="$(find icart_mini_description)/urdf/sensors/hokuyo.urdf.xacro"/>
   <xacro:sensor_hokuyo name="hokuyo" parent="base_link">
-    <origin xyz="0.374295 0 0.2185" rpy="0 0 0"/>
+    <origin xyz="0.12 0 0.3" rpy="0 0 0"/>
   </xacro:sensor_hokuyo>
 </robot>

Commit message: fix: base_linkの位置とキャスターの記述を修正

File: orne_or_description/urdf/cart/orne_or_cart.urdf.xacro (robot description, xacro)
@@ -9,5 +9,5 @@
   <link name="base_link">
     <inertial>
-      <origin xyz="0.030 0 0.0" rpy="0 0 0"/>
+      <origin xyz="-0.3 0 0.2" rpy="0 0 0"/>
       <mass value="25.0"/>
       <inertia ixx="1.0" ixy="0.0" ixz="0.0" iyy="1.0" iyz="0.0" izz="0.1" />
@@ -96,4 +96,10 @@
       <material name="red"/>
     </visual>
+        <collision>
+      <origin xyz="0 0.150 0" rpy="${PI/2} 0 0"/>
+      <geometry>
+        <cylinder length="0.025" radius="0.050"/>
+      </geometry>
+    </collision>
     <visual>
       <origin xyz="0 -0.150 0" rpy="${PI/2} 0 0"/>
@@ -103,10 +109,4 @@
       <material name="red"/>
     </visual>
-    <collision>
-      <origin xyz="0 0.150 0" rpy="${PI/2} 0 0"/>
-      <geometry>
-        <cylinder length="0.025" radius="0.050"/>
-      </geometry>
-    </collision>
     <collision>
       <origin xyz="0 -0.150 0" rpy="${PI/2} 0 0"/>
